File: PRTGN_v1/PRTGN_v1.kicad_pcb (KiCad board)
At the start: 2 copper layers, 56.5 x 86.5 mm, 75 parts, among them IC1 TPS565242DRLR, J1 Barrel_Jack, J2 Screw_Terminal_01x02, J3 Conn_02x08_Odd_Even, J4 Screw_Terminal_01x02, J5 USB_TypeC, J6 Conn_02x08_Odd_Even, J8 Conn_02x08_Odd_Even, J9 Conn_02x08_Odd_Even, M1 Fan_4pin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

Commit message: pcb update
Parts:
- removed C3: 100nF, Capacitor_SMD:C_0805_2012Metric_Pad1.18x1.45mm_HandSolder
- removed J6: Conn_02x08_Odd_Even, Connector_IDC:IDC-Header_2x08_P2.54mm_Vertical_SMD
- removed JP1: SolderJumper_3_Open, Jumper:SolderJumper-3_P2.0mm_Open_TrianglePad1.0x1.5mm
- removed R10: 10k, Resistor_SMD:R_0805_2012Metric_Pad1.20x1.40mm_HandSolder
- removed R5: 2m, Resistor_SMD:R_0805_2012Metric_Pad1.20x1.40mm_HandSolder
- removed U5: INA226, Package_SO:VSSOP-10_3x3mm_P0.5mm
- J8, J9: footprint Connector_PinSocket_2.54mm:PinSocket_2x08_P2.54mm_Vertical -> Connector_PinSocket_2.54mm:PinSocket_2x08_P2.54mm_Vertical_SMD
- U2: moved to B.Cu
- moved D4 38.7 mm to (33.2, 61.5), turned to -90 degrees
- moved R4 38.1 mm to (33.2, 61.0), turned to -90 degrees
- moved D3 37.7 mm to (30.8, 61.5), turned to -90 degrees
- moved R3 36.9 mm to (30.8, 61.0), turned to -90 degrees
- moved M1 29.5 mm to (62.5, 38.0)
- moved M2 29.5 mm to (75.6, 38.0)
- moved TP7 25.0 mm to (84.2, 70.2)
- moved R6 15.6 mm to (92.5, 82.0)
- moved R7 15.6 mm to (92.5, 80.0)
- moved R13 14.8 mm to (68.0, 101.5), turned to -90 degrees
- moved R8 9.83 mm to (65.8, 88.0), turned to 180 degrees
- moved C17 8.89 mm to (83.0, 56.2)
- moved J9 8.86 mm to (45.8, 56.0)
- moved J8 8.50 mm to (84.5, 56.0)
- moved J3 8.00 mm to (65.2, 49.8)
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Connections:
- J3 pad 10: B1 -> B_A
- J3 pad 11: C1 -> C_A
- J3 pad 12: D1 -> D_A
- J3 pad 9: A1 -> A_A
- J8 pad 10: COL_5_A -> COL_3_A
- J8 pad 11: ROW_6_A -> ROW_5_A
- J8 pad 12: COL_6_A -> COL_7_A
- J8 pad 13: ROW_7_A -> ROW_8_A
- J8 pad 14: COL_7_A -> COL_5_A
- J8 pad 15: ROW_8_A -> ROW_4_A
- J8 pad 16: COL_8_A -> COL_1_A
- J8 pad 2: COL_1_A -> COL_2_A
- J8 pad 3: ROW_2_A -> ROW_6_A
- J8 pad 4: COL_2_A -> COL_6_A
- J8 pad 5: ROW_3_A -> ROW_2_A
- J8 pad 6: COL_3_A -> COL_8_A
- J8 pad 7: ROW_4_A -> ROW_7_A
- J8 pad 9: ROW_5_A -> ROW_3_A
- J9 pad 10: COL_5_B -> COL_3_B
- J9 pad 11: ROW_6_B -> ROW_5_B
- J9 pad 12: COL_6_B -> COL_7_B
- J9 pad 13: ROW_7_B -> ROW_8_B
- J9 pad 14: COL_7_B -> COL_5_B
- J9 pad 15: ROW_8_B -> ROW_4_B
- J9 pad 16: COL_8_B -> COL_1_B
- J9 pad 2: COL_1_B -> COL_2_B
- J9 pad 3: ROW_2_B -> ROW_6_B
- J9 pad 4: COL_2_B -> COL_6_B
- J9 pad 5: ROW_3_B -> ROW_2_B
- J9 pad 6: COL_3_B -> COL_8_B
- J9 pad 7: ROW_4_B -> ROW_7_B
- J9 pad 9: ROW_5_B -> ROW_3_B
- Q2 pad 2: VBATT_SHUNT -> VBATT
- R9 pad 1: VBATT_SHUNT -> VBATT
- U1 pad 10: unconnected-(U1-IO17-Pad10) -> LAT2
- U1 pad 11: unconnected-(U1-IO18-Pad11) -> D_B
- U1 pad 12: unconnected-(U1-IO8-Pad12) -> B_B
- U1 pad 23: unconnected-(U1-IO21-Pad23) -> R4
- U1 pad 24: unconnected-(U1-IO47-Pad24) -> B3
- U1 pad 25: unconnected-(U1-IO48-Pad25) -> R3
- U1 pad 28: unconnected-(U1-IO35-Pad28) -> G4
- U1 pad 29: unconnected-(U1-IO36-Pad29) -> G3
- U1 pad 30: unconnected-(U1-IO37-Pad30) -> R2
- U1 pad 31: unconnected-(U1-IO38-Pad31) -> B1
- U1 pad 32: unconnected-(U1-IO39-Pad32) -> R1
- U1 pad 33: unconnected-(U1-IO40-Pad33) -> G1
- U1 pad 34: unconnected-(U1-IO41-Pad34) -> G2
- U1 pad 35: unconnected-(U1-IO42-Pad35) -> B_A
- U1 pad 38: unconnected-(U1-IO2-Pad38) -> D_A
- U1 pad 4: unconnected-(U1-IO4-Pad4) -> CLK1
- U1 pad 5: unconnected-(U1-IO5-Pad5) -> LAT1
- U1 pad 6: unconnected-(U1-IO6-Pad6) -> OE1
- U1 pad 7: unconnected-(U1-IO7-Pad7) -> C_A
- U1 pad 8: unconnected-(U1-IO15-Pad8) -> A_A
- U1 pad 9: unconnected-(U1-IO16-Pad9) -> B2
- U4 pad 12: ~{CS0} -> ~{CS1}
Routing:
- net +5V: track 0.00 -> 176.8 mm, vias 0 -> 7
- net +3V3: track 0.00 -> 60.6 mm, vias 0 -> 3
- net VBUS 5V: track 0.00 -> 41.5 mm, vias 0 -> 2
- net D+: track 0.00 -> 27.0 mm, vias 0 -> 1
- net D-: track 0.00 -> 24.9 mm, vias 0 -> 1
- net COL_4_A: track 0.00 -> 18.8 mm, vias 0 -> 1
- net COL_8_A: track 0.00 -> 18.0 mm, vias 0 -> 1
- net COL_6_A: track 0.00 -> 17.1 mm, vias 0 -> 1
- net COL_5_A: track 0.00 -> 17.0 mm, vias 0 -> 1
- net COL_2_A: track 0.00 -> 16.4 mm, vias 0 -> 1
- net COL_7_A: track 0.00 -> 16.4 mm, vias 0 -> 1
- net COL_1_A: track 0.00 -> 16.3 mm, vias 0 -> 1
- net COL_3_A: track 0.00 -> 15.9 mm, vias 0 -> 1
- net ROW_4_B: track 0.00 -> 14.6 mm, vias 0 -> 1
- net ROW_1_B: track 0.00 -> 14.3 mm, vias 0 -> 1
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- added copper zone on B.Cu, net +5V
- added copper zone on F.Cu, net +5V
- added copper zone on F.Cu, net Net-(D6-A)
- added copper zone on B.Cu, net VBATT
- added copper zone on B.Cu, net VOUT
- added copper zone on F.Cu, net VOUT
Other:
- copper layers 2 -> 4

Commit message: routing
Parts:
- added R10: 10k, Resistor_SMD:R_0805_2012Metric_Pad1.20x1.40mm_HandSolder, B.Cu at (69.0, 85.8)
- added R5: 10k, Resistor_SMD:R_0805_2012Metric_Pad1.20x1.40mm_HandSolder, B.Cu at (59.5, 90.8)
- BZ1, R8: moved to F.Cu
- TP7, TP8: footprint TestPoint:TestPoint_Pad_1.0x1.0mm -> TestPoint:TestPoint_Pad_D1.0mm
- moved D4 48.3 mm to (80.8, 70.5), turned to 90 degrees
- moved R4 48.3 mm to (80.8, 69.5), turned to 90 degrees
- moved R8 21.5 mm to (72.8, 67.8), turned to 90 degrees
- moved R3 21.5 mm to (49.8, 71.0), turned to 90 degrees
- moved D3 21.0 mm to (49.8, 70.5), turned to 90 degrees
- moved C17 18.2 mm to (65.4, 51.4)
- moved BZ1 16.8 mm to (65.2, 64.0), turned to -90 degrees
- moved C16 13.8 mm to (67.5, 52.0)
- moved C13 13.2 mm to (71.0, 86.9)
- moved SW7 12.2 mm to (80.8, 77.8), turned to -90 degrees
- moved SW5 12.0 mm to (80.8, 90.0)
- moved R21 11.2 mm to (67.5, 55.8), turned to -90 degrees
- moved U3 2.75 mm to (74.5, 55.8), turned to 180 degrees
- moved C1 0.10 mm to (68.9, 90.1)
Connections:
- J8 pad 1: ROW_1_A -> COL_1_A
- J8 pad 10: COL_3_A -> ROW_5_A
- J8 pad 11: ROW_5_A -> COL_6_A
- J8 pad 12: COL_7_A -> ROW_6_A
- J8 pad 13: ROW_8_A -> COL_7_A
- J8 pad 14: COL_5_A -> ROW_7_A
- J8 pad 15: ROW_4_A -> COL_8_A
- J8 pad 16: COL_1_A -> ROW_8_A
- J8 pad 2: COL_2_A -> ROW_1_A
- J8 pad 3: ROW_6_A -> COL_2_A
- J8 pad 4: COL_6_A -> ROW_2_A
- J8 pad 5: ROW_2_A -> COL_3_A
- J8 pad 6: COL_8_A -> ROW_3_A
- J8 pad 7: ROW_7_A -> COL_4_A
- J8 pad 8: COL_4_A -> ROW_4_A
- J8 pad 9: ROW_3_A -> COL_5_A
- J9 pad 10: COL_3_B -> COL_5_B
- J9 pad 11: ROW_5_B -> ROW_6_B
- J9 pad 12: COL_7_B -> COL_6_B
- J9 pad 13: ROW_8_B -> ROW_7_B
- J9 pad 14: COL_5_B -> COL_7_B
- J9 pad 15: ROW_4_B -> ROW_8_B
- J9 pad 16: COL_1_B -> COL_8_B
- J9 pad 2: COL_2_B -> COL_1_B
- J9 pad 3: ROW_6_B -> ROW_2_B
- J9 pad 4: COL_6_B -> COL_2_B
- J9 pad 5: ROW_2_B -> ROW_3_B
- J9 pad 6: COL_8_B -> COL_3_B
- J9 pad 7: ROW_7_B -> ROW_4_B
- J9 pad 9: ROW_3_B -> ROW_5_B
- SW6 pad 1: +3V3 -> GND
- SW7 pad 1: +3V3 -> GND
- U1 pad 10: LAT2 -> LED_IO_14
- U1 pad 11: D_B -> unconnected-(U1-IO18-Pad11)
- U1 pad 12: B_B -> unconnected-(U1-IO8-Pad12)
- U1 pad 23: R4 -> unconnected-(U1-IO21-Pad23)
- U1 pad 24: B3 -> unconnected-(U1-IO47-Pad24)
- U1 pad 25: R3 -> unconnected-(U1-IO48-Pad25)
- U1 pad 28: G4 -> LED_IO_21
- U1 pad 29: G3 -> unconnected-(U1-IO36-Pad29)
- U1 pad 30: R2 -> unconnected-(U1-IO37-Pad30)
- U1 pad 31: B1 -> unconnected-(U1-IO38-Pad31)
- U1 pad 32: R1 -> unconnected-(U1-IO39-Pad32)
- U1 pad 33: G1 -> unconnected-(U1-IO40-Pad33)
- U1 pad 34: G2 -> unconnected-(U1-IO41-Pad34)
- U1 pad 35: B_A -> unconnected-(U1-IO42-Pad35)
- U1 pad 38: D_A -> unconnected-(U1-IO2-Pad38)
- U1 pad 39: unconnected-(U1-IO1-Pad39) -> BUTTON_IO_48
- U1 pad 4: CLK1 -> BUTTON_IO_47
- U1 pad 5: LAT1 -> PWM2
- U1 pad 6: OE1 -> PWM1
- U1 pad 7: C_A -> OE1
- U1 pad 8: A_A -> LAT1
- U1 pad 9: B2 -> CLK1
Routing:
- net PWM1: track 0.00 -> 66.0 mm, vias 0 -> 1
- net PWM2: track 0.00 -> 55.7 mm, vias 0 -> 1
- net DOUT: track 0.00 -> 45.5 mm, vias 0 -> 2
- net MOSI: track 0.00 -> 41.3 mm, vias 0 -> 1
- net LAT1: track 1.86 -> 40.7 mm
- net ~{CS1}: track 0.00 -> 33.8 mm, vias 0 -> 3
- net CLK: track 1.61 -> 35.1 mm, vias 1 -> 2
- net ~{CS0}: track 1.86 -> 26.8 mm
- net B_A: track 2.16 -> 26.8 mm, vias 2 -> 1
- net OE1: track 9.77 -> 33.7 mm
- net G2: track 1.78 -> 25.7 mm, vias 2 -> 1
- net G1: track 1.86 -> 24.3 mm, vias 2 -> 1
- net CLK1: track 9.71 -> 31.0 mm
- net D_A: track 3.19 -> 24.2 mm, vias 2 -> 1
- net R2: track 6.05 -> 25.9 mm, vias 2 -> 1
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- added copper zone on B.Cu, net GND
- added copper zone on F.Cu, net GND
