File: PRTGN_v1/PRTGN_v1.kicad_pcb (KiCad board)
At the start: 4 copper layers, 56.5 x 86.5 mm, 73 parts, among them IC1 TPS565242DRLR, J1 Conn_01x06_Pin, J2 Barrel_Jack, J3 Screw_Terminal_01x02, J4 Screw_Terminal_01x02, J5 02x08, J6 USB_TypeC, J7 Conn_02x08_Odd_Even, J8 Conn_02x08_Odd_Even, M1 Fan_4pin, M2 Fan_4pin, Q1 Q_PMOS, Q2 Q_PMOS, SW1 SW_DPDT_x2, SW2 SW_Push, SW3 SW_Push, SW4 SW_Push, SW5 SW_Push, U1 ESP32-S3-WROOM-1, U2 USBLC6-2SC6, U3 MAX7219, U4 MAX7219

Commit message: PCV updates
Parts:
- removed C13, C15: 10uF, Capacitor_Tantalum_SMD:CP_EIA-3216-18_Kemet-A_Pad1.58x1.35mm_HandSolder
- removed C14, C16: 100nF, Capacitor_SMD:C_0805_2012Metric_Pad1.18x1.45mm_HandSolder
- removed Q2: Q_PMOS, Package_TO_SOT_SMD:SOT-23-3
- removed R16, R17, R18, R19, R20: 10k, Resistor_SMD:R_0805_2012Metric_Pad1.20x1.40mm_HandSolder
- removed SW4, SW5: SW_Push, sumec_brd:SW_SPST_EVQPE1
- removed U3, U4: MAX7219, Package_SO:SOP-24_7.5x15.4mm_P1.27mm
- added RN1: YC248-JR-0710KL, sumec-remote_library:resistor_array, F.Cu at (144.3, 61.5)
- added TP4: TestPoint, TestPoint:TestPoint_Pad_D1.0mm, F.Cu at (159.5, 81.0)
- added TP5: TestPoint, TestPoint:TestPoint_Pad_D1.0mm, F.Cu at (159.5, 84.0)
- BZ1: footprint Schrack_brd:BUZZER_CUI_CPT -> gps-compass_brd:CEM-1203_Buzzer; moved to F.Cu
- C1, C2, C6, C7, IC1, L1, U2: moved to F.Cu
- C11, C12: footprint Capacitor_SMD:C_0805_2012Metric_Pad1.18x1.45mm_HandSolder -> Capacitor_SMD:C_0805_2012Metric; moved to F.Cu
- C3, C5: value 22uF -> 100nF; footprint Capacitor_Tantalum_SMD:CP_EIA-2012-12_Kemet-R_Pad1.30x1.05mm_HandSolder -> Capacitor_SMD:C_0805_2012Metric_Pad1.18x1.45mm_HandSolder; moved to F.Cu
- C4, C8: value 100nF -> 22uF; footprint Capacitor_SMD:C_0805_2012Metric_Pad1.18x1.45mm_HandSolder -> Capacitor_Tantalum_SMD:CP_EIA-2012-12_Kemet-R_Pad1.30x1.05mm_HandSolder; moved to F.Cu
- D1, D2: value LED -> D_Schottky; footprint LED_SMD:LED_0805_2012Metric_Pad1.15x1.40mm_HandSolder -> Diode_SMD:D_1206_3216Metric_Pad1.42x1.75mm_HandSolder
- D5, D6: value D_Schottky -> LED; footprint Diode_SMD:D_1206_3216Metric_Pad1.42x1.75mm_HandSolder -> LED_SMD:LED_0805_2012Metric_Pad1.15x1.40mm_HandSolder
- H1, H2, H3, H4: value Mounting Hole M2 -> Mounting Hole M3; footprint MountingHole:MountingHole_2.2mm_M2_Pad_Via -> MountingHole:MountingHole_3.2mm_M3_Pad_Via
- J1: value Conn_01x06_Pin -> USB_TypeC; footprint Connector_PinSocket_2.54mm:PinSocket_2x03_P2.54mm_Vertical_SMD -> sumec_brd:HRO_TYPE-C-31-M-12
- J5: value 02x08 -> Conn_01x05_Socket; footprint Connector_IDC:IDC-Header_2x08_P2.54mm_Vertical_SMD -> Connector_Wire:SolderWire-0.5sqmm_1x05_P4.6mm_D0.9mm_OD2.1mm_Relief
- J6: value USB_TypeC -> Conn_01x05_Socket; footprint sumec_brd:HRO_TYPE-C-31-M-12 -> Connector_Wire:SolderWire-0.5sqmm_1x05_P4.6mm_D0.9mm_OD2.1mm_Relief
- J7: value Conn_02x08_Odd_Even -> 02x08; footprint Connector_PinSocket_2.54mm:PinSocket_2x08_P2.54mm_Vertical_SMD -> Connector_IDC:IDC-Header_2x08_P2.54mm_Vertical_SMD
- J8: value Conn_02x08_Odd_Even -> Conn_01x03_Socket; footprint Connector_PinSocket_2.54mm:PinSocket_2x08_P2.54mm_Vertical_SMD -> Connector_Wire:SolderWire-0.5sqmm_1x03_P4.6mm_D0.9mm_OD2.1mm_Relief
- R1, R2: value 560R -> 10k; moved to F.Cu
- R10: value 45k -> 10k; footprint Resistor_SMD:R_0805_2012Metric_Pad1.20x1.40mm_HandSolder -> Resistor_SMD:R_0805_2012Metric; moved to F.Cu
- R11: value 10k -> 2.2k; moved to F.Cu
- R12: value 100k -> 2.2k
- R13, R14: value 15R -> 220R
- R15: value 10k -> 0R; footprint Resistor_SMD:R_0805_2012Metric_Pad1.20x1.40mm_HandSolder -> Resistor_SMD:R_0805_2012Metric; moved to F.Cu
- R3: value 220R -> 100k; moved to F.Cu
- R4: value 220R -> 45k; moved to F.Cu
- R5: value 0R -> 10k; moved to F.Cu
- R6, R7: value 10k -> 15R; moved to F.Cu
- R9: footprint Resistor_SMD:R_0805_2012Metric_Pad1.20x1.40mm_HandSolder -> Resistor_SMD:R_0805_2012Metric; moved to F.Cu
- moved J5 123.2 mm to (188.2, 42.1)
- moved J6 122.7 mm to (165.2, 23.3), turned to -90 degrees
- moved H2 99.4 mm to (125.0, 85.2), turned to 0 degrees
- moved D3 98.6 mm to (146.8, 88.1), turned to 0 degrees
- moved C12 92.0 mm to (140.2, 93.9), turned to 0 degrees
- moved J7 87.7 mm to (133.4, 54.8)
- moved D2 86.7 mm to (117.2, 44.9), turned to 0 degrees
- moved J8 86.1 mm to (170.2, 46.8)
- moved H4 85.6 mm to (125.0, 101.2)
- moved R15 85.2 mm to (156.1, 88.0), turned to 0 degrees
- moved BZ1 85.0 mm to (151.4, 80.0), turned to 0 degrees
- moved SW3 84.0 mm to (133.5, 97.0), turned to 0 degrees
- moved D5 81.0 mm to (146.8, 94.2), turned to 0 degrees
- moved D1 80.0 mm to (117.2, 41.5), turned to 0 degrees
- moved TP3 79.8 mm to (159.5, 77.9), turned to 0 degrees
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Connections:
- C11 pad 1: EN -> GND
- C11 pad 2: GND -> EN
- C12 pad 1: BOOT -> GND
- C12 pad 2: GND -> BOOT
- C3 pad 1: +5V -> GND
- C3 pad 2: GND -> /POWER/SHLD
- C5 pad 1: +3V3 -> +5V
- C9 pad 1: GND -> +3V3
- C9 pad 2: /CONNECTORS/SHLD -> GND
- D1 pad 2: VBUS 5V -> VBATT
- D2 pad 1: Net-(D2-K) -> Net-(D1-K)
- D2 pad 2: VOUT -> VBUS_5V
- D3 pad 2: LED_IO_35 -> VBATT
- D4 pad 2: LED_IO_08 -> VBUS_5V
- D5 pad 1: +5V -> Net-(D5-K)
- D5 pad 2: Net-(D5-A) -> LED_IO_35
- D6 pad 1: +5V -> Net-(D6-K)
- D6 pad 2: VBUS 5V -> LED_IO_08
- J5 pad 1: R1 -> EXP_SW_1
- J5 pad 2: G1 -> EXP_SW_2
- J5 pad 3: B1 -> EXP_SW_3
- J5 pad 4: GND -> EXP_SW_4
- J5 pad 5: R2 -> GND
- J7 pad 1: ROW_1_B -> R1
- J7 pad 10: COL_5_B -> B
- J7 pad 11: ROW_6_B -> C
- J7 pad 12: COL_6_B -> D
- J7 pad 13: ROW_7_B -> CLK_75
- J7 pad 14: COL_7_B -> LAT
- J7 pad 15: ROW_8_B -> OE
- J7 pad 16: COL_8_B -> GND
- J7 pad 2: COL_1_B -> G1
- J7 pad 3: ROW_2_B -> B1
- J7 pad 4: COL_2_B -> GND
- J7 pad 5: ROW_3_B -> R2
- J7 pad 6: COL_3_B -> G2
- J7 pad 7: ROW_4_B -> B2
- J7 pad 8: COL_4_B -> GND
- J7 pad 9: ROW_5_B -> A
- J8 pad 1: COL_1_A -> +3V3
- J8 pad 2: ROW_1_A -> MTH_SW
- J8 pad 3: COL_2_A -> GND
- M1 pad 3: TACHO1 -> unconnected-(M1-Tacho-Pad3)
- M2 pad 3: TACHO2 -> unconnected-(M2-Tacho-Pad3)
- Q1 pad 1: VBUS 5V -> /POWER/FET_SW
- Q1 pad 2: VOUT -> Net-(D1-K)
- Q1 pad 3: Net-(D5-A) -> +5V
- R1 pad 1: Net-(D1-K) -> IO_FREE_36
- R1 pad 2: GND -> +3V3
- R10 pad 1: +3V3 -> BOOT
- R10 pad 2: FB -> +3V3
- R11 pad 1: FB -> Net-(D3-K)
- R12 pad 1: /CONNECTORS/SHLD -> Net-(D4-K)
- R13 pad 1: D+ IN -> Net-(D5-K)
- R13 pad 2: Net-(R13-Pad2) -> GND
- R14 pad 1: D- IN -> Net-(D6-K)
- R14 pad 2: Net-(R14-Pad2) -> GND
- R15 pad 1: EN -> BZ_PWM
- R15 pad 2: +3V3 -> Net-(BZ1-+)
- R2 pad 1: Net-(D2-K) -> IO_FREE_23
- R2 pad 2: GND -> +3V3
- R3 pad 1: Net-(D3-K) -> /POWER/SHLD
- R4 pad 1: Net-(D4-K) -> +3V3
- R4 pad 2: GND -> FB
- R5 pad 1: BZ_PWM -> FB
- R5 pad 2: Net-(BZ1-+) -> GND
- R6 pad 1: IO_FREE_36 -> D+ IN
- R6 pad 2: +3V3 -> Net-(R6-Pad2)
- R7 pad 1: IO_FREE_23 -> D- IN
- R7 pad 2: +3V3 -> Net-(R7-Pad2)
- R8 pad 1: VBUS 5V -> Net-(D1-K)
- R8 pad 2: GND -> /POWER/FET_SW
- R9 pad 1: VBATT -> EN
- R9 pad 2: /POWER/FET_SW -> +3V3
- SW3 pad 2: BTN_IO_01 -> BOOT
- TP3 pad 1: +3V3 -> unconnected-(TP3-Pad1)
- U1 pad 12: LED_IO_08 -> EXP_SW_6
- U1 pad 17: CLK -> EXP_SW_3
- U1 pad 24: IO_FREE_47 -> EXP_SW_8
- U1 pad 25: IO_FREE_48 -> EXP_SW_7
- U1 pad 35: ~{CS1} -> IO_FREE_36
- U1 pad 39: BTN_IO_01 -> EXP_SW_4
- U1 pad 4: BTN_IO_04 -> EXP_SW_5
- U1 pad 5: ~{CS0} -> EXP_SW_1
- U1 pad 6: MOSI -> EXP_SW_2
- U1 pad 7: FAN1_PWM -> MTH_SW
- U1 pad 8: FAN2_PWM -> unconnected-(U1-IO15-Pad8)
- U2 pad 1: Net-(R13-Pad2) -> Net-(R6-Pad2)
- U2 pad 3: Net-(R14-Pad2) -> Net-(R7-Pad2)
Routing:
- net +5V: track 172.1 -> 0.00 mm, vias 7 -> 0
- net +3V3: track 86.2 -> 0.00 mm, vias 4 -> 0
- net FAN2_PWM: track 63.4 -> 0.00 mm, vias 1 -> 0
- net FAN1_PWM: track 53.1 -> 0.00 mm, vias 1 -> 0
- net ~{CS1}: track 49.1 -> 0.00 mm, vias 4 -> 0
- net G1: track 43.4 -> 0.00 mm, vias 2 -> 0
- net IO_FREE_36: track 42.9 -> 0.00 mm, vias 4 -> 0
- net MOSI: track 41.9 -> 0.00 mm, vias 2 -> 0
- net G2: track 41.7 -> 0.00 mm, vias 2 -> 0
- net VBUS 5V: track 41.5 -> 0.00 mm, vias 2 -> 0
- net CLK: track 39.9 -> 0.00 mm, vias 3 -> 0
- net R2: track 38.8 -> 0.00 mm, vias 2 -> 0
- net LAT: track 38.1 -> 0.00 mm, vias 2 -> 0
- net IO_FREE_23: track 36.8 -> 0.00 mm, vias 2 -> 0
- net DOUT: track 36.5 -> 0.00 mm, vias 2 -> 0
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- removed copper zone on B.Cu, net +5V
- removed copper zone on F.Cu, net +5V
- removed copper zone on In2.Cu, net +5V
- removed copper zone on B.Cu, net /CONNECTORS/SHLD
- removed copper zone on F.Cu, net /CONNECTORS/SHLD
- removed copper zone on B.Cu, net GND
- removed copper zone on F.Cu, net GND
- removed copper zone on F.Cu, net Net-(D5-A)
- removed copper zone on B.Cu, net VBATT
- removed copper zone on B.Cu, net VOUT
- removed copper zone on F.Cu, net VOUT
Other:
- board outline removed
- board text removed: "3V3"
- board text removed: "48 47 36 23 3V3 GND"
- board text removed: "5V"
- board text removed: "BOOT"
- board text removed: "FAN1"
- board text removed: "FAN2"
- board text removed: "GND"
- board text removed: "IO01"
- board text removed: "IO04"
- board text removed: "IO08"
- board text removed: "IO35"
- board text removed: "PWR"
- board text removed: "RST"
- board text removed: "USB"

Commit message: pcb layout.
Parts:
- added J9: APDS-9960, Connector_Wire:SolderWire-0.5sqmm_1x04_P4.6mm_D0.9mm_OD2.1mm, F.Cu at (162.6, 84.8)
- J7: value 02x08 -> 02x08 IDC
- moved J8 141.4 mm to (48.0, 118.1)
- moved J2 105.6 mm to (183.3, 118.0), turned to 90 degrees
- moved RN1 99.2 mm to (63.1, 118.5)
- moved H4 83.2 mm to (185.1, 43.5)
- moved C2 77.3 mm to (68.8, 145.6)
- moved C1 77.3 mm to (69.5, 136.6)
- moved R1 77.3 mm to (68.8, 139.6)
- moved R2 77.3 mm to (68.8, 142.6)
- moved J7 62.8 mm to (78.7, 24.0)
- moved J5 61.9 mm to (128.6, 58.5), turned to -90 degrees
- moved U1 60.6 mm to (148.3, 50.1)
- moved H3 60.0 mm to (185.1, 92.1)
- moved J6 53.7 mm to (168.0, 77.0), turned to 90 degrees
- moved J1 53.6 mm to (139.0, 94.0)
- moved M1 52.9 mm to (99.4, 119.2)
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Connections:
- net IO_FREE_23 renamed SCL
- R1 pad 1: IO_FREE_36 -> SDA
- U1 pad 28: LED_IO_35 -> SDA
- U1 pad 29: IO_FREE_36 -> LED_IO_35
- U1 pad 35: IO_FREE_36 -> IO42
- U1 pad 8: unconnected-(U1-IO15-Pad8) -> ADC2_IO15
Other:
- board outline added: 80 x 55 mm
- board text added: "what rotation should hub75 be?"

Commit message: PCB
Parts:
- added J10: JST-VH4, Connector_JST:JST_VH_B4P-VH-B_1x04_P3.96mm_Vertical, F.Cu at (156.5, 90.0)
- added J11: JST-VH4, Connector_JST:JST_VH_B4P-VH-B_1x04_P3.96mm_Vertical, F.Cu at (138.1, 90.0)
- J5, J6: footprint Connector_Wire:SolderWire-0.5sqmm_1x05_P4.6mm_D0.9mm_OD2.1mm_Relief -> gps-compass_brd:SolderWire-Relief-5pin
- J8: footprint Connector_Wire:SolderWire-0.5sqmm_1x03_P4.6mm_D0.9mm_OD2.1mm_Relief -> gps-compass_brd:SolderWire-Relief-3pin
- J9: footprint Connector_Wire:SolderWire-0.5sqmm_1x04_P4.6mm_D0.9mm_OD2.1mm -> gps-compass_brd:SolderWire-Relief-4pin
- moved BZ1 266.1 mm to (-33.0, -96.0)
- moved J8 151.6 mm to (183.1, 49.3), turned to 180 degrees
- moved RN1 124.2 mm to (173.5, 61.5), turned to 180 degrees
- moved SW2 110.0 mm to (168.2, 46.5), turned to 180 degrees
- moved SW3 108.7 mm to (168.2, 53.3), turned to 180 degrees
- moved M2 96.3 mm to (186.8, 86.6), turned to 90 degrees
- moved J4 89.9 mm to (188.0, 93.8), turned to 180 degrees
- moved IC1 86.6 mm to (63.9, 134.8)
- moved J7 71.3 mm to (135.0, 67.8)
- moved SW1 70.4 mm to (153.2, 78.0), turned to 90 degrees
- moved C7 55.5 mm to (75.0, 139.8)
- moved C8 55.5 mm to (75.0, 142.6)
- moved C9 55.5 mm to (72.9, 123.8)
- moved R4 55.5 mm to (73.5, 149.8)
- moved R5 55.5 mm to (62.9, 123.7)
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Other:
- board size 80 x 55 mm -> 90 x 55 mm

Commit message: layout PCB etc
Parts:
- moved BZ1 257.5 mm to (172.2, 59.5), turned to -90 degrees
- moved R2 157.7 mm to (215.0, 43.5)
- moved R1 157.2 mm to (215.0, 41.5)
- moved R4 127.4 mm to (171.9, 68.9), turned to 90 degrees
- moved C8 124.6 mm to (174.9, 68.2)
- moved IC1 124.3 mm to (172.0, 73.5), turned to 90 degrees
- moved C7 121.9 mm to (174.9, 70.0)
- moved R5 120.3 mm to (170.1, 68.9), turned to -90 degrees
- moved C6 119.3 mm to (174.9, 71.8)
- moved C9 113.7 mm to (174.9, 73.7)
- moved C4 111.2 mm to (170.1, 76.5), turned to -90 degrees
- moved R10 110.3 mm to (170.2, 50.8)
- moved C5 108.4 mm to (170.1, 72.7), turned to 90 degrees
- moved L1 108.2 mm to (173.3, 76.5)
- moved C2 102.3 mm to (142.4, 48.4), turned to 90 degrees
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Connections:
- C10 pad 1: VBUS 5V -> VBUS_5V
- U2 pad 5: VBUS 5V -> VBUS_5V
Routing:
- net D- IN: track 0.00 -> 6.24 mm
- net D+ IN: track 0.00 -> 5.46 mm

Commit message: pcb silksdnree neded
Parts:
- removed H1, H2, H3, H4: Mounting Hole M3, MountingHole:MountingHole_3.2mm_M3_Pad_Via
- removed the J2 at (176.5, 82.5)
- removed RN1: YC248-JR-0710KL, sumec-remote_library:resistor_array
- added J3: SOLDER PAD, PRTGN_brd:SolderWirePad_1x01_SMD, B.Cu at (182.8, 103.8)
- added J4: SOLDER PAD, PRTGN_brd:SolderWirePad_1x01_SMD, B.Cu at (127.8, 103.8)
- added TP6: TestPoint, TestPoint:TestPoint_Pad_D1.0mm, B.Cu at (161.8, 47.5)
- BZ1: footprint gps-compass_brd:CEM-1203_Buzzer -> inset:AST0827MW-03BTRQ_MAL
- C1: value 10uF -> 100nF; footprint Capacitor_Tantalum_SMD:CP_EIA-3216-18_Kemet-A_Pad1.58x1.35mm_HandSolder -> Capacitor_SMD:C_0805_2012Metric
- C10, C2, C3, C5, C9: footprint Capacitor_SMD:C_0805_2012Metric_Pad1.18x1.45mm_HandSolder -> Capacitor_SMD:C_0805_2012Metric
- C4, C6, C7, C8: footprint Capacitor_Tantalum_SMD:CP_EIA-2012-12_Kemet-R_Pad1.30x1.05mm_HandSolder -> Capacitor_Tantalum_SMD:CP_EIA-2012-12_Kemet-R
- D1, D2: footprint Diode_SMD:D_1206_3216Metric_Pad1.42x1.75mm_HandSolder -> Diode_SMD:D_2114_3652Metric
- D3, D4, D5, D6: footprint LED_SMD:LED_0805_2012Metric_Pad1.15x1.40mm_HandSolder -> LED_SMD:LED_0805_2012Metric
- J6: renamed from J3; footprint TerminalBlock:TerminalBlock_Xinya_XY308-2.54-2P_1x02_P2.54mm_Horizontal -> TerminalBlock_Phoenix:TerminalBlock_Phoenix_MKDS-1,5-2-5.08_1x02_P5.08mm_Horizontal
- J7: renamed from J4; footprint TerminalBlock:TerminalBlock_Xinya_XY308-2.54-2P_1x02_P2.54mm_Horizontal -> TerminalBlock_Phoenix:TerminalBlock_Phoenix_MKDS-1,5-2-5.08_1x02_P5.08mm_Horizontal
- R1, R11, R12, R13, R14, R2, R3, R4, R5, R6, R7, R8: footprint Resistor_SMD:R_0805_2012Metric_Pad1.20x1.40mm_HandSolder -> Resistor_SMD:R_0805_2012Metric
- SW1: value SW_DPDT_x2 -> SW_SPDT
- TP1: footprint sumec_graphic:SPS_LOGO_IMG -> TestPoint:TestPoint_Pad_D1.0mm
- TP5: moved to B.Cu
- U2: footprint Package_TO_SOT_SMD:TSOT-23-6_HandSoldering -> Package_TO_SOT_SMD:TSOT-23-6
- moved TP1 499.7 mm to (182.8, 93.3), turned to 0 degrees
- moved TP2 101.6 mm to (127.5, 106.5)
- moved R14 63.9 mm to (166.8, 51.1)
- moved R13 59.0 mm to (166.8, 53.1)
- moved R2 56.5 mm to (168.2, 75.3), turned to 180 degrees
- moved D6 56.4 mm to (178.4, 59.1), turned to 180 degrees
- moved M2 56.3 mm to (130.8, 92.8), turned to 0 degrees
- moved R1 55.7 mm to (168.2, 71.8), turned to 180 degrees
- moved M1 55.0 mm to (171.3, 92.8), turned to 0 degrees
- moved TP5 53.8 mm to (159.5, 47.5), turned to -90 degrees
- moved TP4 52.3 mm to (161.0, 67.8)
- moved TP3 51.8 mm to (167.2, 79.0), turned to 90 degrees
- moved D5 51.2 mm to (178.4, 61.3), turned to 180 degrees
- moved J11 48.8 mm to (171.5, 75.3), turned to 90 degrees
- moved J5 47.7 mm to (119.2, 46.2), turned to -45 degrees
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- renumbered J7 to J10, J9 to J11, J8 to J12, J10 to J2, J11 to J5, J5 to J8, J6 to J9
Connections:
- D5 pad 1: Net-(D5-K) -> GND
- D5 pad 2: LED_IO_35 -> Net-(D5-A)
- D6 pad 1: Net-(D6-K) -> GND
- D6 pad 2: LED_IO_08 -> Net-(D6-A)
- M1 pad 4: FAN2_PWM -> unconnected-(M1-PWM-Pad4)
- M2 pad 4: FAN1_PWM -> unconnected-(M2-PWM-Pad4)
- R13 pad 1: Net-(D5-K) -> LED_IO_42
- R13 pad 2: GND -> Net-(D5-A)
- R14 pad 1: Net-(D6-K) -> LED_IO_02
- R14 pad 2: GND -> Net-(D6-A)
- TP2 pad 1: +5V -> GND
- TP3 pad 1: unconnected-(TP3-Pad1) -> +3V3
- TP4 pad 1: +3V3 -> FREE_IO
- TP5 pad 1: unconnected-(TP5-Pad1) -> UART_RX
- U1 pad 10: LAT -> EXP_SW_6
- U1 pad 11: CLK_75 -> EXP_SW_7
- U1 pad 12: EXP_SW_6 -> EXP_SW_8
- U1 pad 17: EXP_SW_3 -> G2
- U1 pad 18: D -> A
- U1 pad 19: C -> B
- U1 pad 20: A -> C
- U1 pad 21: B2 -> D
- U1 pad 22: B -> CLK_75
- U1 pad 23: SCL -> LAT
- U1 pad 24: EXP_SW_8 -> OE
- U1 pad 25: EXP_SW_7 -> FREE_IO
- U1 pad 29: LED_IO_35 -> SCL
- U1 pad 30: R2 -> MTH_SW
- U1 pad 31: B1 -> EXP_SW_1
- U1 pad 32: G2 -> EXP_SW_2
- U1 pad 33: R1 -> EXP_SW_3
- U1 pad 34: G1 -> EXP_SW_4
- U1 pad 35: IO42 -> LED_IO_42
- U1 pad 36: unconnected-(U1-IO44-Pad36) -> UART_RX
- U1 pad 37: unconnected-(U1-IO43-Pad37) -> UART_TX
- U1 pad 38: BZ_PWM -> LED_IO_02
- U1 pad 39: EXP_SW_4 -> BZ_PWM
- U1 pad 4: EXP_SW_5 -> G1
- U1 pad 5: EXP_SW_1 -> R1
- U1 pad 6: EXP_SW_2 -> B1
- U1 pad 7: MTH_SW -> R2
- U1 pad 8: ADC2_IO15 -> B2
- U1 pad 9: OE -> EXP_SW_5
Routing:
- net +5V: track 0.00 -> 185.6 mm, vias 0 -> 17
- net GND: track 0.00 -> 110.0 mm, vias 0 -> 47
- net +3V3: track 0.00 -> 90.8 mm, vias 0 -> 6
- net EXP_SW_1: track 0.00 -> 54.8 mm
- net EXP_SW_4: track 0.00 -> 54.3 mm
- net EXP_SW_2: track 0.00 -> 53.8 mm
- net EXP_SW_3: track 0.00 -> 52.8 mm
- net BOOT: track 0.00 -> 52.1 mm, vias 0 -> 2
- net EXP_SW_5: track 0.00 -> 48.8 mm
- net EXP_SW_6: track 0.00 -> 44.8 mm
- net VBUS_5V: track 0.00 -> 44.4 mm, vias 0 -> 8
- net EXP_SW_7: track 0.00 -> 41.6 mm
- net EXP_SW_8: track 0.00 -> 39.6 mm
- net OE: track 0.00 -> 38.7 mm, vias 0 -> 2
- net CLK_75: track 0.00 -> 35.1 mm, vias 0 -> 2
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- added copper zone on F.Cu, net +3V3
- added copper zone on F.Cu, net +5V
- added copper zone on B.Cu, net GND
- added copper zone on F.Cu, net Net-(D1-K)
- added copper zone on F.Cu, net Net-(IC1-SW)
- added copper zone on B.Cu, net VBATT
- added copper zone on B.Cu, net VBUS_5V
Other:
- board size 90 x 55 mm -> 85 x 70 mm
- board text added: "what rotation should hub75 be? check pinouts of everything"
- board text removed: "what rotation should hub75 be?"

Commit message: final
Parts:
- moved TP2 2.79 mm to (125.0, 107.5)
- moved D6 0.06 mm to (178.4, 59.1)
Connections:
- J8 pad 1: EXP_SW_1 -> EXP_SW_5
- J8 pad 2: EXP_SW_2 -> EXP_SW_6
- J8 pad 3: EXP_SW_3 -> EXP_SW_7
- J8 pad 4: EXP_SW_4 -> EXP_SW_8
- J9 pad 1: EXP_SW_5 -> EXP_SW_1
- J9 pad 2: EXP_SW_6 -> EXP_SW_2
- J9 pad 3: EXP_SW_7 -> EXP_SW_3
- J9 pad 4: EXP_SW_8 -> EXP_SW_4
- U1 pad 10: EXP_SW_6 -> EXP_SW_2
- U1 pad 11: EXP_SW_7 -> EXP_SW_3
- U1 pad 12: EXP_SW_8 -> EXP_SW_4
- U1 pad 31: EXP_SW_1 -> EXP_SW_5
- U1 pad 32: EXP_SW_2 -> EXP_SW_6
- U1 pad 33: EXP_SW_3 -> EXP_SW_7
- U1 pad 34: EXP_SW_4 -> EXP_SW_8
- U1 pad 9: EXP_SW_5 -> EXP_SW_1
Routing:
- net EXP_SW_8: track 39.6 -> 54.3 mm
- net EXP_SW_4: track 54.3 -> 39.6 mm
- net EXP_SW_7: track 41.6 -> 52.8 mm
- net EXP_SW_3: track 52.8 -> 41.6 mm
- net EXP_SW_6: track 44.8 -> 53.8 mm
- net EXP_SW_2: track 53.8 -> 44.8 mm
- net D-: track 26.4 -> 32.8 mm
- net EXP_SW_5: track 48.8 -> 54.8 mm
- net EXP_SW_1: track 54.8 -> 48.8 mm
- net D+: track 25.9 -> 31.1 mm
- net GND: track 110.0 -> 109.1 mm
Other:
- board text added: "02"
- board text added: "3V3"
- board text added: "42"
- board text added: "5V"
- board text added: "BEEEP :3"
- board text added: "BOOP"
- board text added: "BOOT"
- board text added: "EXPRESSION SW"
- board text added: "GND"
- board text added: "IO48"
- board text added: "MAIN DISPLAYS"
- board text added: "MOUTH"
- board text added: "MTH"
- board text added: "NEG-"
- board text added: "POS+"
- board text added: "RST"
- board text added: "SCL"
- board text added: "SDA"
- board text added: "SW1"
- board text added: "SW2"
- board text added: "SW3"
- board text added: "SW4"
- board text added: "SW5"
- board text added: "SW6"
- board text added: "SW7"
- board text added: "SW8"
- board text added: "USB"
- board text added: "VBATT"
- board text added: "d+ 51,77 = 19.77 + 32 D- 48,01 = 14.47 + 33.54 d+ 30, 30 d- 30.9, 32.54"

Commit message: prtgnd
Parts:
- added G***: LOGO, LOGO, F.Cu at (159.8, 74.2)
- added TPd1: TestPoint, PRTGN_brd:APERTURE_ART, B.Cu at (153.4, 72.0)
- added TPd3: TestPoint, sumec_graphic:BOYKISSER_IMG, F.Cu at (157.0, 83.6)
- added TPd6: TestPoint, sumec_graphic:OWO_IMG, F.Cu at (155.2, 64.5)
- added TPd8: TestPoint, sumec_graphic:PURO_CHANGED_IMG, F.Cu at (126.2, 90.0)
Connections:
- U2 pad 1: Net-(R6-Pad2) -> Net-(R7-Pad2)
- U2 pad 3: Net-(R7-Pad2) -> Net-(R6-Pad2)
- U2 pad 4: D- -> D+
- U2 pad 6: D+ -> D-
Routing:
- net D-: track 32.8 -> 29.6 mm, vias 2 -> 0
- net D+: track 31.1 -> 28.7 mm
- net Net-(R7-Pad2): track 11.7 -> 14.1 mm
- net Net-(R6-Pad2): track 16.7 -> 14.8 mm
Other:
- copper layers 4 -> 2
- board text added: "PRTGN BOARD V1"
- board text added: "WHAT'S THIS?"
- board text added: "You like making PCBs, don't you?"
- board text added: "made by bismarx"
- board text removed: "d+ 51,77 = 19.77 + 32 D- 48,01 = 14.47 + 33.54 d+ 30, 30 d- 30.9, 32.54"

Commit message: prtoogen visdor silkscreenm - order
Parts:
- added TPd2: TestPoint, PRTGN_brd:LEGOSHI_SILK, F.Cu at (155.2, 75.8)
- added TPd4: TestPoint, sumec_graphic:OWO_IMG, B.Cu at (141.8, 47.3)
- TPd3: moved to B.Cu
- moved TPd8 64.2 mm to (171.6, 44.6), turned to 180 degrees
- moved G*** 35.8 mm to (141.5, 43.5)
- moved TPd1 13.3 mm to (155.8, 59.0), turned to -168 degrees
- moved TPd3 5.32 mm to (162.2, 84.6), turned to 180 degrees
- moved D3 0.86 mm to (184.3, 105.2)
- moved R11 0.86 mm to (182.3, 105.2)
Routing:
- net GND: track 109.1 -> 110.9 mm
- net VBATT: track 27.9 -> 28.7 mm
Other:
- board text added: "A"
- board text added: "B"
- board text added: "B1"
- board text added: "B2"
- board text added: "C"
- board text added: "CLK"
- board text added: "D"
- board text added: "G1"
- board text added: "G2"
- board text added: "LAT"
- board text added: "MAIN DISPL."
- board text added: "OE"
- board text added: "PROOOOOOOOT :3"
- board text added: "R1"
- board text added: "R2"
- board text added: "RX"
- board text added: "TX"
- board text added: "VBAT"
- board text removed: "MAIN DISPLAYS"
- board text removed: "VBATT"
- board text removed: "what rotation should hub75 be? check pinouts of everything"
