File: PRTGN_v1/connectors.kicad_sch (KiCad schematic)
At the start: 11 parts, among them J3 Conn_02x08_Odd_Even, J5 USB_TypeC, J6 Conn_02x08_Odd_Even, M1 Fan_4pin, M2 Fan_4pin, U2 USBLC6-2SC6

Commit message: pcb update
Parts:
- removed J6: Conn_02x08_Odd_Even, Connector_IDC:IDC-Header_2x08_P2.54mm_Vertical_SMD, symbol Connector_Generic:Conn_02x08_Odd_Even
Connections:
- net B1: no longer J3.10 (Pin_10)
- net A1 renamed A_A
- net C1 renamed C_A
- net D1 renamed D_A
- new net B_A: J3.10 (Pin_10)

Commit message: upd
Parts:
- J5: renamed from J3; value Conn_02x08_Odd_Even -> 02x08
- renumbered C12 to C10, C11 to C9, J5 to J6, R17 to R12, R18 to R13, R19 to R14
Connections:
- net A_A renamed A
- net B_A renamed B
- net CLK1 renamed CLK_75
- net C_A renamed C
- net D_A renamed D
- net LAT1 renamed LAT
- net OE1 renamed OE
- net PWM1 renamed FAN2_PWM
- net PWM2 renamed FAN1_PWM
Other:
- note added: "HUB-75"
- note removed: "HUB-75 RGB LED MATRIX CONN"
- moved on the sheet: C10, C9, J5, J6, M1, M2, R12, R13, R14, U2
