File: PRTGN_v1/mechanics.kicad_sch (KiCad schematic)
At the start: 13 parts, among them SW5 SW_Push, SW6 SW_Push, SW7 SW_Push, SW8 SW_Push

Commit message: routing
Parts:
- added R10, R5: 10k, Resistor_SMD:R_0805_2012Metric_Pad1.20x1.40mm_HandSolder, symbol Device:R
- TP7, TP8: footprint TestPoint:TestPoint_Pad_1.0x1.0mm -> TestPoint:TestPoint_Pad_D1.0mm
Connections:
- net +3V3: now also R10.2, R5.2; no longer SW6.1, SW7.1
- net BUTTON_IO_47: now also R10.1
- net BUTTON_IO_48: now also R5.1
- net GND: now also SW6.1, SW7.1
Other:
- note added: "INPUT_PULLUP"

Commit message: upd
Parts:
- added R20: 10k, Resistor_SMD:R_0805_2012Metric_Pad1.20x1.40mm_HandSolder, symbol Device:R
- renumbered C13 to C11, C14 to C12, R20 to R15, R5 to R16, R10 to R17, SW5 to SW2, SW6 to SW3, SW7 to SW4, SW8 to SW5, TP7 to TP2, TP8 to TP3
Connections:
- net +3V3: now also R20.2
- net BOOT: now also R20.1
- net BUTTON_IO_47 renamed BTN_IO_04
- net BUTTON_IO_48 renamed BTN_IO_01
Other:
- note removed: "EN=RESET, BOOT=bootloader mode Enable (EN) is the 3.3V regulator's enable pin. It's pulled up, so connect to ground to disable the 3.3V regulator. This means that you can use this pin connected to a pushbutton to restart your ESP32, for example."
- note removed: "INPUT_PULLUP"
- moved on the sheet: C11, C12, H1, H2, H3, H4, R15, R16, R17, SW2, SW3, SW4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
