File: PRTGN_v1/power.kicad_sch (KiCad schematic)
At the start: 25 parts, among them IC1 TPS565242DRLR, J1 Barrel_Jack, J2 Screw_Terminal_01x02, J4 Screw_Terminal_01x02, Q1 Q_PMOS, Q2 Q_PMOS, SW1 SW_DPDT_x2, U5 INA226

Commit message: pcb update
Parts:
- removed C3: 100nF, Capacitor_SMD:C_0805_2012Metric_Pad1.18x1.45mm_HandSolder, symbol Device:C
- removed JP1: SolderJumper_3_Open, Jumper:SolderJumper-3_P2.0mm_Open_TrianglePad1.0x1.5mm, symbol Jumper:SolderJumper_3_Open
- removed R10: 10k, Resistor_SMD:R_0805_2012Metric_Pad1.20x1.40mm_HandSolder, symbol Device:R
- removed R5: 2m, Resistor_SMD:R_0805_2012Metric_Pad1.20x1.40mm_HandSolder, symbol Device:R
- removed U5: INA226, Package_SO:VSSOP-10_3x3mm_P0.5mm, symbol Sensor_Energy:INA226
Connections:
- net VBATT_SHUNT is gone; now on net VBATT: Q2.2 (S), R9.1
Other:
- note removed: "I2C adress = 0x40"
- note removed: "VOLTAGE READING"

Commit message: upd
Parts:
- renumbered C5 to C3, C6 to C4, C7 to C5, C8 to C6, C9 to C7, C10 to C8, D6 to D5, D7 to D6, J1 to J2, J2 to J3, R15 to R10, R16 to R11, R13 to R8
Other:
- note added: "5V TERMINAL"
- note added: "BARREL JACK"
- note removed: "5V SCREW TERMINAL"
- note removed: "BARREL JACK CONN"
- note removed: "FeedBack voltage divider, usinf formula from datasheet 45.3 in reality? check before ordering."
- moved on the sheet: C3, C4, C5, C6, C7, C8, D5, D6, IC1, J2, J3, J4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
