File: PRTGN_v1/matrix.kicad_sch (KiCad schematic)
At the start: 10 parts, among them J8 Conn_02x08_Odd_Even, J9 Conn_02x08_Odd_Even, U3 MAX7219, U4 MAX7219

Commit message: pcb update
Parts:
- J8, J9: footprint Connector_PinSocket_2.54mm:PinSocket_2x08_P2.54mm_Vertical -> Connector_PinSocket_2.54mm:PinSocket_2x08_P2.54mm_Vertical_SMD
Connections:
- net COL_1_A: now also J8.16 (Pin_16); no longer J8.2 (Pin_2)
- net COL_1_B: now also J9.16 (Pin_16); no longer J9.2 (Pin_2)
- net COL_2_A: now also J8.2 (Pin_2); no longer J8.4 (Pin_4)
- net COL_2_B: now also J9.2 (Pin_2); no longer J9.4 (Pin_4)
- net COL_3_A: now also J8.10 (Pin_10); no longer J8.6 (Pin_6)
- net COL_3_B: now also J9.10 (Pin_10); no longer J9.6 (Pin_6)
- net COL_5_A: now also J8.14 (Pin_14); no longer J8.10 (Pin_10)
- net COL_5_B: now also J9.14 (Pin_14); no longer J9.10 (Pin_10)
- net COL_6_A: now also J8.4 (Pin_4); no longer J8.12 (Pin_12)
- net COL_6_B: now also J9.4 (Pin_4); no longer J9.12 (Pin_12)
- net COL_7_A: now also J8.12 (Pin_12); no longer J8.14 (Pin_14)
- net COL_7_B: now also J9.12 (Pin_12); no longer J9.14 (Pin_14)
- net COL_8_A: now also J8.6 (Pin_6); no longer J8.16 (Pin_16)
- net COL_8_B: now also J9.6 (Pin_6); no longer J9.16 (Pin_16)
- net ROW_2_A: now also J8.5 (Pin_5); no longer J8.3 (Pin_3)
- net ROW_2_B: now also J9.5 (Pin_5); no longer J9.3 (Pin_3)
- net ROW_3_A: now also J8.9 (Pin_9); no longer J8.5 (Pin_5)
- net ROW_3_B: now also J9.9 (Pin_9); no longer J9.5 (Pin_5)
- net ROW_4_A: now also J8.15 (Pin_15); no longer J8.7 (Pin_7)
- net ROW_4_B: now also J9.15 (Pin_15); no longer J9.7 (Pin_7)
- net ROW_5_A: now also J8.11 (Pin_11); no longer J8.9 (Pin_9)
- net ROW_5_B: now also J9.11 (Pin_11); no longer J9.9 (Pin_9)
- net ROW_6_A: now also J8.3 (Pin_3); no longer J8.11 (Pin_11)
- net ROW_6_B: now also J9.3 (Pin_3); no longer J9.11 (Pin_11)
- net ROW_7_A: now also J8.7 (Pin_7); no longer J8.13 (Pin_13)
- net ROW_7_B: now also J9.7 (Pin_7); no longer J9.13 (Pin_13)
- net ROW_8_A: now also J8.13 (Pin_13); no longer J8.15 (Pin_15)
- net ROW_8_B: now also J9.13 (Pin_13); no longer J9.15 (Pin_15)
- net ~{CS0}: no longer U4.12 (LOAD)
- new net ~{CS1}: U4.12 (LOAD)

Commit message: routing
Connections:
- net COL_1_A: now also J8.1 (Pin_1); no longer J8.16 (Pin_16)
- net COL_1_B: now also J9.2 (Pin_2); no longer J9.16 (Pin_16)
- net COL_2_A: now also J8.3 (Pin_3); no longer J8.2 (Pin_2)
- net COL_2_B: now also J9.4 (Pin_4); no longer J9.2 (Pin_2)
- net COL_3_A: now also J8.5 (Pin_5); no longer J8.10 (Pin_10)
- net COL_3_B: now also J9.6 (Pin_6); no longer J9.10 (Pin_10)
- net COL_4_A: now also J8.7 (Pin_7); no longer J8.8 (Pin_8)
- net COL_5_A: now also J8.9 (Pin_9); no longer J8.14 (Pin_14)
- net COL_5_B: now also J9.10 (Pin_10); no longer J9.14 (Pin_14)
- net COL_6_A: now also J8.11 (Pin_11); no longer J8.4 (Pin_4)
- net COL_6_B: now also J9.12 (Pin_12); no longer J9.4 (Pin_4)
- net COL_7_A: now also J8.13 (Pin_13); no longer J8.12 (Pin_12)
- net COL_7_B: now also J9.14 (Pin_14); no longer J9.12 (Pin_12)
- net COL_8_A: now also J8.15 (Pin_15); no longer J8.6 (Pin_6)
- net COL_8_B: now also J9.16 (Pin_16); no longer J9.6 (Pin_6)
- net ROW_1_A: now also J8.2 (Pin_2); no longer J8.1 (Pin_1)
- net ROW_2_A: now also J8.4 (Pin_4); no longer J8.5 (Pin_5)
- net ROW_2_B: now also J9.3 (Pin_3); no longer J9.5 (Pin_5)
- net ROW_3_A: now also J8.6 (Pin_6); no longer J8.9 (Pin_9)
- net ROW_3_B: now also J9.5 (Pin_5); no longer J9.9 (Pin_9)
- net ROW_4_A: now also J8.8 (Pin_8); no longer J8.15 (Pin_15)
- net ROW_4_B: now also J9.7 (Pin_7); no longer J9.15 (Pin_15)
- net ROW_5_A: now also J8.10 (Pin_10); no longer J8.11 (Pin_11)
- net ROW_5_B: now also J9.9 (Pin_9); no longer J9.11 (Pin_11)
- net ROW_6_A: now also J8.12 (Pin_12); no longer J8.3 (Pin_3)
- net ROW_6_B: now also J9.11 (Pin_11); no longer J9.3 (Pin_3)
- net ROW_7_A: now also J8.14 (Pin_14); no longer J8.7 (Pin_7)
- net ROW_7_B: now also J9.13 (Pin_13); no longer J9.7 (Pin_7)
- net ROW_8_A: now also J8.16 (Pin_16); no longer J8.13 (Pin_13)
- net ROW_8_B: now also J9.15 (Pin_15); no longer J9.13 (Pin_13)
Other:
- moved on the sheet: J8, J9

Commit message: upd
Parts:
- renumbered C15 to C13, C16 to C14, C17 to C15, C18 to C16, J9 to J7, R21 to R18, R22 to R19
Other:
- note added: "8x8 MATRIX CONN"
- note added: "MAX7219"
- moved on the sheet: C13, C14, C15, C16, J7, J8, R18, R19, U3, U4

Commit message: pcb updates
Parts:
- J7, J8: footprint Connector_PinSocket_2.54mm:PinSocket_2x08_P2.54mm_Vertical_SMD -> Connector_PinSocket_2.54mm:PinSocket_2x08_P2.54mm_Vertical
Changed lines of the file:
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@@
 			)
 		)
-		(property "Footprint" "Connector_PinSocket_2.54mm:PinSocket_2x08_P2.54mm_Vertical_SMD"
+		(property "Footprint" "Connector_PinSocket_2.54mm:PinSocket_2x08_P2.54mm_Vertical"
 			(at 116.84 156.21 0)
 			(effects
@@
 			)
 		)
-		(property "Datasheet" "~"
+		(property "Datasheet" "]"
 			(at 116.84 156.21 0)
 			(effects
@@
 			)
 		)
-		(property "Footprint" "Connector_PinSocket_2.54mm:PinSocket_2x08_P2.54mm_Vertical_SMD"
+		(property "Footprint" "Connector_PinSocket_2.54mm:PinSocket_2x08_P2.54mm_Vertical"
 			(at 81.28 156.21 0)
 			(effects
