File: PRTGN_v1/mcu.kicad_sch (KiCad schematic)
At the start: 15 parts, among them U1 ESP32-S3-WROOM-1

Commit message: pcb update
Connections:
- net R2: now reaches U1.30 (IO37)
- net B1: now reaches U1.31 (IO38)
- net R1: now reaches U1.32 (IO39)
- net G1: now reaches U1.33 (IO40)
- net G2: now reaches U1.34 (IO41)
- net B_A: now reaches U1.35 (IO42)
- net D_A: now reaches U1.38 (IO2)
- net CLK1: now reaches U1.4 (IO4)
- net LAT1: now reaches U1.5 (IO5)
- net OE1: now reaches U1.6 (IO6)
- net C_A: now reaches U1.7 (IO7)
- net A_A: now reaches U1.8 (IO15)
- net B2: now reaches U1.9 (IO16)
- no-connect marks 2 -> 5

Commit message: routing
Connections:
- net A_A: no longer U1.8 (IO15)
- net B1: no longer U1.31 (IO38)
- net B2: no longer U1.9 (IO16)
- net BUTTON_IO_47: now also U1.4 (IO4)
- net BUTTON_IO_48: now also U1.39 (IO1)
- net B_A: no longer U1.35 (IO42)
- net CLK1: now also U1.9 (IO16); no longer U1.4 (IO4)
- net C_A: no longer U1.7 (IO7)
- net D_A: no longer U1.38 (IO2)
- net G1: no longer U1.33 (IO40)
- net G2: no longer U1.34 (IO41)
- net LAT1: now also U1.8 (IO15); no longer U1.5 (IO5)
- net LED_IO_14: now also U1.10 (IO17)
- net LED_IO_21: now also U1.28 (IO35)
- net OE1: now also U1.7 (IO7); no longer U1.6 (IO6)
- net PWM1: now also U1.6 (IO6)
- net PWM2: now also U1.5 (IO5)
- net R1: no longer U1.32 (IO39)
- net R2: no longer U1.30 (IO37)

Commit message: upd
Parts:
- renumbered R8 to R5
Connections:
- net BZ_IO02 is gone; now on net BZ_PWM: R5.1
- net PWM1 is gone; now on net MOSI: U1.6 (IO6)
- net PWM2 is gone; now on net ~{CS0}: U1.5 (IO5)
- net SCL is gone; now on net IO_FREE_23: R7.1
- net SDA is gone; now on net IO_FREE_36: R6.1
- net B1: now also U1.31 (IO38)
- net B2: now also U1.21 (IO13)
- net G1: now also U1.34 (IO41)
- net G2: now also U1.32 (IO39)
- net R1: now also U1.33 (IO40)
- net R2: now also U1.30 (IO37)
- net ~{CS1}: now also U1.35 (IO42)
- net CLK_75: now reaches U1.11 (IO18)
- net LED_IO_08: now reaches U1.12 (IO8)
- net LED_IO_08: now also D4.2 (A)
- net CLK: now reaches U1.17 (IO9)
- net D: now reaches U1.18 (IO10)
- net C: now reaches U1.19 (IO11)
- net A: now reaches U1.20 (IO12)
- net B: now reaches U1.22 (IO14)
- net IO_FREE_23: now reaches U1.23 (IO21)
- net IO_FREE_47: now reaches U1.24 (IO47)
- net IO_FREE_48: now reaches U1.25 (IO48)
- net IO_FREE_36: now reaches U1.29 (IO36)
- net BZ_PWM: now reaches U1.38 (IO2)
- net BUTTON_IO_47 renamed BTN_IO_04
- net BUTTON_IO_48 renamed BTN_IO_01
- net CLK1 renamed OE
- net LAT1 renamed FAN2_PWM
- net LED_IO_14 renamed LAT
- net LAT: no longer D4.2 (A)
- net LED_IO_21 renamed LED_IO_35
- net OE1 renamed FAN1_PWM
Other:
- note removed: "jumpers clock - HUB75"
- moved on the sheet: BZ1, C1, C2, D1, D2, D3, D4, R1, R2, R3, R4, R5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

Commit message: pcb updates
Parts:
- BZ1: footprint Schrack_brd:BUZZER_CUI_CPT -> gps-compass_brd:CEM-1203_Buzzer
- R5: footprint Resistor_SMD:R_0805_2012Metric_Pad1.20x1.40mm_HandSolder -> Resistor_SMD:R_0805_2012Metric; LCSC (none) -> C17633
Other:
- note added: "AUDIO"
- note removed: "BUZZER"
