File: PRTGN_v1/PRTGN_v1.kicad_sch (KiCad schematic)
At the start: 1 part

Commit message: PCV updates
Other:
- sheet CONNECTORS renamed FUNCTIONS
- removed sheet 8X8 MATRIX
- added sheet DEBUG (sub-sch/debug.kicad_sch)
- sheet FUNCTIONS: file connectors.kicad_sch -> sub-sch/functions.kicad_sch
- sheet MCU: file mcu.kicad_sch -> sub-sch/mcu.kicad_sch
- sheet MECHANICS: file mechanics.kicad_sch -> sub-sch/mechanics.kicad_sch
- sheet POWER: file power.kicad_sch -> sub-sch/power.kicad_sch

Commit message: PCB
Other:
- note added: "ALIEXPRESS DISPLAY"
- note added: "JST VH CONN AND HOUSING"
- note added: "JST VH4 CABLE"
Changed lines of the file:
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@@
+		)
+	)
+	(text "JST VH4 CABLE"
+		(exclude_from_sim no)
+		(at 79.375 130.175 0)
+		(effects
+			(font
+				(size 1.27 1.27)
+				(italic yes)
+			)
+			(href "https://www.aliexpress.com/item/1005005097178659.html?spm=a2g0o.productlist.main.1.3f962028cCI2oB&algo_pvid=0ec6399e-4c12-40aa-bfe5-ad70e34caf19&algo_exp_id=0ec6399e-4c12-40aa-bfe5-ad70e34caf19-0&pdp_ext_f=%7B\"order\"%3A\"8\"%2C\"eval\"%3A\"1\"%7D&pdp_npi=6%40dis%21USD%211.57%211.08%21%21%211.57%211.08%21%402103867617544229092177424e8429%2112000031647173870%21sea%21CZ%216186796272%21X%211%210%21&curPageLogUid=BJkgc1dDGujU&utparam-url=scene%3Asearch%7Cquery_from%3A")
+		)
+	)
+	(text "ALIEXPRESS DISPLAY"
+		(exclude_from_sim no)
+		(at 80.645 121.285 0)
+		(effects
+			(font
+				(size 1.27 1.27)
+				(italic yes)
+			)
+			(href "https://www.aliexpress.com/item/1005003258372186.html?spm=a2g0o.productlist.main.6.2b8164c6VVgrJZ&algo_pvid=f2ff8835-5b5e-48e1-ab17-aeadfc1f4b31&algo_exp_id=f2ff8835-5b5e-48e1-ab17-aeadfc1f4b31-5&pdp_ext_f=%7B\"order\"%3A\"80\"%2C\"eval\"%3A\"1\"%7D&pdp_npi=6%40dis%21USD%2117.62%218.81%21%21%2117.62%218.81%21%402103891017544204332836938ede21%2112000024890032393%21sea%21CZ%210%21ABX%211%210%21&curPageLogUid=6hwtcY8OWy5e&utparam-url=scene%3Asearch%7Cquery_from%3A#nav-description")
 		)
 	)
@@
 		)
 	)
+	(text "JST VH CONN AND HOUSING"
+		(exclude_from_sim no)
+		(at 80.645 124.46 0)
+		(effects
+			(font
+				(size 1.27 1.27)
+				(italic yes)
+			)
+			(href "https://www.aliexpress.com/item/1005006867575378.html?src=google&pdp_npi=4%40dis!USD!1.11!0.76!!!!!%40!12000038566059650!ppc!!!&src=google&albch=shopping&acnt=615-992-9880&isdl=y&slnk=&plac=&mtctp=&albbt=Google_7_shopping&aff_platform=google&aff_short_key=_oFgTQeV&gclsrc=aw.ds&&albagn=888888&&ds_e_adid=&ds_e_matchtype=&ds_e_device=c&ds_e_network=x&ds_e_product_group_id=&ds_e_product_id=en1005006867575378&ds_e_product_merchant_id=107917273&ds_e_product_country=CZ&ds_e_product_language=en&ds_e_product_channel=online&ds_e_product_store_id=&ds_url_v=2&albcp=22479481823&albag=&isSmbAutoCall=false&needSmbHouyi=false&gad_source=1&gad_campaignid=22482954463&gclid=Cj0KCQjw18bEBhCBARIsAKuAFEaDuYjB2BdZjFun25MXcafKrZBwwFhnyjbScrGbarbSoFRxSw7wIAcaAtPkEALw_wcB")
+		)
+	)

Commit message: pcb silksdnree neded
Parts:
- TPd1: renamed from TP1; footprint sumec_graphic:SPS_LOGO_IMG -> (none)
Changed lines of the file:
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@@
 		)
-	)
-	(junction
-		(at 86.36 173.99)
-		(diameter 0)
-		(color 0 0 0 0)
-	)
-	(junction
-		(at 97.79 173.99)
-		(diameter 0)
-		(color 0 0 0 0)
-	)
-	(junction
-		(at 90.17 173.99)
-		(diameter 0)
-		(color 0 0 0 0)
-	)
-	(junction
-		(at 93.98 173.99)
-		(diameter 0)
-		(color 0 0 0 0)
-	)
-	(junction
-		(at 101.6 173.99)
-		(diameter 0)
-		(color 0 0 0 0)
 	)
 	(no_connect
@@
 	(wire
 		(pts
-			(xy 93.98 171.45) (xy 93.98 173.99)
-		)
-		(stroke
-			(width 0)
-			(type default)
-		)
-	)
-	(wire
-		(pts
-			(xy 93.98 173.99) (xy 97.79 173.99)
-		)
-		(stroke
-			(width 0)
-			(type default)
-		)
-	)
-	(wire
-		(pts
-			(xy 86.36 173.99) (xy 90.17 173.99)
-		)
-		(stroke
-			(width 0)
-			(type default)
-		)
-	)
-	(wire
-		(pts
-			(xy 90.17 173.99) (xy 93.98 173.99)
-		)
-		(stroke
-			(width 0)
-			(type default)
-		)
-	)
-	(wire
-		(pts
-			(xy 86.36 171.45) (xy 86.36 173.99)
-		)
-		(stroke
-			(width 0)
-			(type default)
-		)
-	)
-	(wire
-		(pts
-			(xy 101.6 173.99) (xy 105.41 173.99)
-		)
-		(stroke
-			(width 0)
-			(type default)
-		)
-	)
-	(wire
-		(pts
-			(xy 90.17 173.99) (xy 90.17 171.45)
-		)
-		(stroke
-			(width 0)
-			(type default)
-		)
-	)
-	(wire
-		(pts
-			(xy 101.6 173.99) (xy 101.6 171.45)
-		)
-		(stroke
-			(width 0)
-			(type default)
-		)
-	)
-	(wire
-		(pts
-			(xy 97.79 173.99) (xy 101.6 173.99)
-		)
-		(stroke
-			(width 0)
-			(type default)
-		)
-	)
-	(wire
-		(pts
-			(xy 86.36 173.99) (xy 86.36 177.8)
-		)
-		(stroke
-			(width 0)
-			(type default)
-		)
-	)
-	(wire
-		(pts
-			(xy 97.79 171.45) (xy 97.79 173.99)
-		)
-		(stroke
-			(width 0)
-			(type default)
-		)
-	)
-	(wire
-		(pts
-			(xy 105.41 171.45) (xy 105.41 173.99)
+			(xy 86.36 171.45) (xy 86.36 177.8)
 		)
 		(stroke
@@
 		(dnp no)
 		(fields_autoplaced yes)
-		(property "Reference" "TP1"
+		(property "Reference" "TPd1"
 			(at 88.9 166.8779 0)
 			(effects
@@
 			)
 		)
-		(property "Footprint" "sumec_graphic:SPS_LOGO_IMG"
+		(property "Footprint" ""
 			(at 91.44 171.45 0)
 			(effects
@@
 			(project "PRTGN_v1"
 				(path "/4072676c-cfd2-418d-bd22-dac92e3db49a"
-					(reference "TP1")
+					(reference "TPd1")
 					(unit 1)
 				)
@@
 	)
 	(sheet
-		(at 55.88 80.01)
-		(size 48.26 25.4)
+		(at 52.705 80.01)
+		(size 55.88 27.305)
 		(exclude_from_sim no)
 		(in_bom yes)
@@
 		)
 		(property "Sheetname" "MCU"
-			(at 55.88 79.2984 0)
+			(at 52.705 79.2984 0)
 			(effects
 				(font
@@
 		)
 		(property "Sheetfile" "sub-sch/mcu.kicad_sch"
-			(at 55.88 105.9946 0)
+			(at 52.705 107.8996 0)
 			(effects
 				(font
@@
 	)
 	(sheet
-		(at 118.11 39.37)
-		(size 55.88 27.94)
+		(at 117.475 39.37)
+		(size 57.15 27.94)
 		(exclude_from_sim no)
 		(in_bom yes)
@@
 		)
 		(property "Sheetname" "MECHANICS"
-			(at 118.11 38.6584 0)
+			(at 117.475 38.6584 0)
 			(effects
 				(font
@@
 		)
 		(property "Sheetfile" "sub-sch/mechanics.kicad_sch"
-			(at 118.11 67.8946 0)
+			(at 117.475 67.8946 0)
 			(effects
 				(font
@@
 	(sheet
 		(at 117.475 78.74)
-		(size 55.88 27.94)
-		(exclude_from_sim no)
-		(in_bom yes)
+		(size 57.15 27.94)
+		(exclude_from_sim no)
+		(in_bom yes)

Commit message: prtgnd
Parts:
- added TPd3: TestPoint, sumec_graphic:BOYKISSER_IMG, symbol Connector:TestPoint
- added TPd6: TestPoint, sumec_graphic:OWO_IMG, symbol Connector:TestPoint
- added TPd7: TestPoint, sumec_graphic:BLAHAJ_IMG_silk, symbol Connector:TestPoint
- added TPd8: TestPoint, sumec_graphic:PURO_CHANGED_IMG, symbol Connector:TestPoint
- TPd1: footprint (none) -> PRTGN_brd:APERTURE_ART
Connections:
- no-connect marks 1 -> 5
Other:
- note removed: "SPS LOGO"

Commit message: didnt close it
Parts:
- removed TPd7: TestPoint, sumec_graphic:BLAHAJ_IMG_silk, symbol Connector:TestPoint
Connections:
- no-connect marks 5 -> 4
Changed lines of the file:
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@@
-	)
-	(no_connect
-		(at 104.14 170.18)
 	)
 	(no_connect
@@
 	(wire
 		(pts
-			(xy 104.14 168.91) (xy 104.14 170.18)
+			(xy 99.06 168.91) (xy 99.06 170.18)
 		)
 		(stroke
@@
 		)
 	)
-	(wire
-		(pts
-			(xy 99.06 168.91) (xy 99.06 170.18)
-		)
-		(stroke
-			(width 0)
-			(type default)
-		)
-	)
 	(symbol
 		(lib_id "Connector:TestPoint")
-		(at 104.14 168.91 0)
+		(at 99.06 168.91 0)
 		(unit 1)
 		(exclude_from_sim no)
@@
 		(fields_autoplaced yes)
 		(property "Reference" "TPd8"
-			(at 106.68 164.3379 0)
+			(at 101.6 164.3379 0)
 			(effects
 				(font
@@
 		)
 		(property "Value" "TestPoint"
-			(at 106.68 166.8779 0)
+			(at 101.6 166.8779 0)
 			(effects
 				(font
@@
 		)
 		(property "Footprint" "sumec_graphic:PURO_CHANGED_IMG"
-			(at 109.22 168.91 0)
+			(at 104.14 168.91 0)
 			(effects
 				(font
@@
 		)
 		(property "Datasheet" "~"
-			(at 109.22 168.91 0)
+			(at 104.14 168.91 0)
 			(effects
 				(font
@@
 		)
 		(property "Description" "test point"
-			(at 104.14 168.91 0)
+			(at 99.06 168.91 0)
 			(effects
 				(font
@@
 					(unit 1)
 				)
-			)
-		)
-	)
-	(symbol
-		(lib_id "Connector:TestPoint")
-		(at 99.06 168.91 0)
-		(unit 1)
-		(exclude_from_sim no)
-		(in_bom yes)
-		(on_board yes)
-		(dnp no)
-		(fields_autoplaced yes)
-		(property "Reference" "TPd7"
-			(at 101.6 164.3379 0)
-			(effects
-				(font
-					(size 1.27 1.27)
-				)
-				(justify left)
-				(hide yes)
-			)
-		)
-		(property "Value" "TestPoint"
-			(at 101.6 166.8779 0)
-			(effects
-				(font
-					(size 1.27 1.27)
-				)
-				(justify left)
-				(hide yes)
-			)
-		)
-		(property "Footprint" "sumec_graphic:BLAHAJ_IMG_silk"
-			(at 104.14 168.91 0)
-			(effects
-				(font
-					(size 1.27 1.27)
-				)
-				(hide yes)
-			)
-		)
-		(property "Datasheet" "~"
-			(at 104.14 168.91 0)
-			(effects
-				(font
-					(size 1.27 1.27)
-				)
-				(hide yes)
-			)
-		)
-		(property "Description" "test point"
-			(at 99.06 168.91 0)
-			(effects
-				(font
-					(size 1.27 1.27)
-				)
-				(hide yes)
-			)
-		)
-		(pin "1"
-		)
-		(instances
-			(project "PRTGN_v1"
-				(path "/4072676c-cfd2-418d-bd22-dac92e3db49a"
-					(reference "TPd7")
-					(unit 1)
-				)

Commit message: prtoogen visdor silkscreenm - order
Parts:
- added TPd2: TestPoint, PRTGN_brd:LEGOSHI_SILK, symbol Connector:TestPoint
- added TPd4: TestPoint, sumec_graphic:OWO_IMG, symbol Connector:TestPoint
Connections:
- no-connect marks 4 -> 6
