File: PRTGN_v1/sub-sch/debug.kicad_sch (KiCad schematic)
At the start: 14 parts

Commit message: pcb silksdnree neded
Parts:
- added TP4, TP6: TestPoint, TestPoint:TestPoint_Pad_D1.0mm, symbol Connector:TestPoint
- BZ1: footprint gps-compass_brd:CEM-1203_Buzzer -> inset:AST0827MW-03BTRQ_MAL
- D3, D4, D5, D6: footprint LED_SMD:LED_0805_2012Metric_Pad1.15x1.40mm_HandSolder -> LED_SMD:LED_0805_2012Metric
- R11, R12, R13, R14: footprint Resistor_SMD:R_0805_2012Metric_Pad1.20x1.40mm_HandSolder -> Resistor_SMD:R_0805_2012Metric
- renumbered TP2 to TP1, TP3 to TP2, TP4 to TP3
Connections:
- net GND: now also D5.1 (K), D6.1 (K), TP2.1; no longer R13.2, R14.2
- net LED_IO_42: now reaches R13.1
- net LED_IO_42: no longer D5.1 (K)
- net UART_RX: now reaches TP5.1
- net LED_IO_02: now reaches R14.1
- net LED_IO_02: no longer D6.1 (K)
- net LED_IO_08: no longer names the net of D6.2 (A)
- net LED_IO_08: now also R14.2
- net LED_IO_35: no longer names the net of D5.2 (A)
- net LED_IO_35: now also R13.2
- new net FREE_IO: TP4.1
- new net UART_TX: TP6.1
Other:
- moved on the sheet: D5, D6, R13, R14, TP1, TP2, TP3
