File: PRTGN_v1/sub-sch/mechanics.kicad_sch (KiCad schematic)
At the start: 12 parts, among them M1 Fan_4pin, M2 Fan_4pin, SW2 SW_Push, SW3 SW_Push

Commit message: pcb silksdnree neded
Parts:
- removed H1, H2, H3, H4: Mounting Hole M3, MountingHole:MountingHole_3.2mm_M3_Pad_Via, symbol Mechanical:MountingHole_Pad
Connections:
- net FAN1_PWM: no longer names the net of M2.4 (PWM)
- net FAN2_PWM: no longer names the net of M1.4 (PWM)
- no-connect marks 2 -> 4
Other:
- note removed: "M3 Padded Mounting holes"
- note removed: "MOUNTING"
- moved on the sheet: C11, C12, M1, M2, R10, R9, SW2, SW3
