File: PRTGN_v1/sub-sch/functions.kicad_sch (KiCad schematic)
At the start: 6 parts, among them J5 Conn_01x05_Socket, J6 Conn_01x05_Socket, J7 02x08 IDC, J8 Conn_01x03_Socket, J9 APDS-9960

Commit message: pcb layout.
Parts:
- J9: footprint (none) -> Connector_Wire:SolderWire-0.5sqmm_1x04_P4.6mm_D0.9mm_OD2.1mm
Other:
- note added: "Connectors for microswitches"
- note added: "HUB75 display connector"
- note added: "IR proximity"
- note added: "Reed switch"
Changed lines of the file:
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@@
+		)
+	)
+	(text "IR proximity"
+		(exclude_from_sim no)
+		(at 181.61 62.865 0)
+		(effects
+			(font
+				(face "Bahnschrift")
+				(size 1 1)
+				(thickness 0.2)
+				(bold yes)
+				(color 0 0 0 1)
+			)
+			(justify left bottom)
 		)
 	)
@@
 		)
 	)
+	(text "HUB75 display connector"
+		(exclude_from_sim no)
+		(at 132.08 63.5 0)
+		(effects
+			(font
+				(face "Bahnschrift")
+				(size 1 1)
+				(thickness 0.2)
+				(bold yes)
+				(color 0 0 0 1)
+			)
+			(justify left bottom)
+		)
+	)
 	(text "HUB-75 DISP."
 		(exclude_from_sim no)
@@
 				(size 5 5)
 				(thickness 1.2)
+				(bold yes)
+				(color 0 0 0 1)
+			)
+			(justify left bottom)
+		)
+	)
+	(text "Reed switch"
+		(exclude_from_sim no)
+		(at 181.61 92.71 0)
+		(effects
+			(font
+				(face "Bahnschrift")
+				(size 1 1)
+				(thickness 0.2)
+				(bold yes)
+				(color 0 0 0 1)
+			)
+			(justify left bottom)
+		)
+	)
+	(text "Connectors for microswitches"
+		(exclude_from_sim no)
+		(at 46.99 62.865 0)
+		(effects
+			(font
+				(face "Bahnschrift")
+				(size 1 1)
+				(thickness 0.2)
 				(bold yes)
 				(color 0 0 0 1)
@@
 			)
 		)
-		(property "Footprint" ""
+		(property "Footprint" "Connector_Wire:SolderWire-0.5sqmm_1x04_P4.6mm_D0.9mm_OD2.1mm"
 			(at 204.47 67.31 0)
 			(effects

Commit message: PCB
Parts:
- J5, J6: footprint Connector_Wire:SolderWire-0.5sqmm_1x05_P4.6mm_D0.9mm_OD2.1mm_Relief -> gps-compass_brd:SolderWire-Relief-5pin
- J8: footprint Connector_Wire:SolderWire-0.5sqmm_1x03_P4.6mm_D0.9mm_OD2.1mm_Relief -> gps-compass_brd:SolderWire-Relief-3pin
- J9: footprint Connector_Wire:SolderWire-0.5sqmm_1x04_P4.6mm_D0.9mm_OD2.1mm -> gps-compass_brd:SolderWire-Relief-4pin
Changed lines of the file:
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@@
 			)
 		)
-		(property "Footprint" "Connector_Wire:SolderWire-0.5sqmm_1x04_P4.6mm_D0.9mm_OD2.1mm"
+		(property "Footprint" "gps-compass_brd:SolderWire-Relief-4pin"
 			(at 204.47 67.31 0)
 			(effects
@@
 			)
 		)
-		(property "Footprint" "Connector_Wire:SolderWire-0.5sqmm_1x05_P4.6mm_D0.9mm_OD2.1mm_Relief"
+		(property "Footprint" "gps-compass_brd:SolderWire-Relief-5pin"
 			(at 71.12 74.93 0)
 			(effects
@@
 			)
 		)
-		(property "Footprint" "Connector_Wire:SolderWire-0.5sqmm_1x03_P4.6mm_D0.9mm_OD2.1mm_Relief"
+		(property "Footprint" "gps-compass_brd:SolderWire-Relief-3pin"
 			(at 205.74 99.06 0)
 			(effects
@@
 			)
 		)
-		(property "Footprint" "Connector_Wire:SolderWire-0.5sqmm_1x05_P4.6mm_D0.9mm_OD2.1mm_Relief"
+		(property "Footprint" "gps-compass_brd:SolderWire-Relief-5pin"
 			(at 71.12 91.44 0)
 			(effects

Commit message: pcb silksdnree neded
Parts:
- removed RN1: YC248-JR-0710KL, sumec-remote_library:resistor_array, symbol SUMEC:YC248-JR-0710KL
- renumbered J7 to J10, J9 to J11, J8 to J12, J5 to J8, J6 to J9
Other:
- moved on the sheet: J10, J11, J12, J8, J9

Commit message: final
Connections:
- net EXP_SW_1: now also J9.1 (Pin_1); no longer J8.1 (Pin_1)
- net EXP_SW_2: now also J9.2 (Pin_2); no longer J8.2 (Pin_2)
- net EXP_SW_3: now also J9.3 (Pin_3); no longer J8.3 (Pin_3)
- net EXP_SW_4: now also J9.4 (Pin_4); no longer J8.4 (Pin_4)
- net EXP_SW_5: now also J8.1 (Pin_1); no longer J9.1 (Pin_1)
- net EXP_SW_6: now also J8.2 (Pin_2); no longer J9.2 (Pin_2)
- net EXP_SW_7: now also J8.3 (Pin_3); no longer J9.3 (Pin_3)
- net EXP_SW_8: now also J8.4 (Pin_4); no longer J9.4 (Pin_4)
