File: PRTGN_v1/sub-sch/mcu.kicad_sch (KiCad schematic)
At the start: 15 parts, among them U1 ESP32-S3-WROOM-1

Commit message: PCV updates
Parts:
- removed BZ1: Buzzer, gps-compass_brd:CEM-1203_Buzzer, symbol Device:Buzzer
- removed D1, D2, D3, D4: LED, LED_SMD:LED_0805_2012Metric_Pad1.15x1.40mm_HandSolder, symbol Device:LED
- removed R1, R2: 560R, Resistor_SMD:R_0805_2012Metric_Pad1.20x1.40mm_HandSolder, symbol Device:R
- removed R3, R4: 220R, Resistor_SMD:R_0805_2012Metric_Pad1.20x1.40mm_HandSolder, symbol Device:R
- removed R5: 0R, Resistor_SMD:R_0805_2012Metric, symbol Device:R
- renumbered R6 to R1, R7 to R2
Connections:
- net LED_IO_35: now also U1.29 (IO36); no longer U1.28 (IO35)
- net BTN_IO_01 renamed EXP_SW_4
- net BTN_IO_04 renamed EXP_SW_5
- net CLK renamed EXP_SW_3
- net FAN1_PWM renamed MTH_SW
- net FAN2_PWM renamed ADC2_IO15
- net IO_FREE_23 renamed SCL
- net IO_FREE_36 renamed SDA
- net SDA: now also U1.28 (IO35); no longer U1.29 (IO36)
- net IO_FREE_47 renamed EXP_SW_8
- net IO_FREE_48 renamed EXP_SW_7
- net LED_IO_08 renamed EXP_SW_6
- net MOSI renamed EXP_SW_2
- net ~{CS0} renamed EXP_SW_1
- net ~{CS1} renamed IO42
Other:
- note removed: "AUDIO"
- note removed: "Battery power"
- note removed: "LED SIGNALISATION"
- note removed: "Status LED1"
- note removed: "Status LED2"
- note removed: "VBUS Power"
- moved on the sheet: C1, C2, R1, R2, U1

Commit message: pcb silksdnree neded
Parts:
- removed C1: 10uF, Capacitor_Tantalum_SMD:CP_EIA-3216-18_Kemet-A_Pad1.58x1.35mm_HandSolder, symbol Device:C_Polarized
- added C1: 100nF, Capacitor_SMD:C_0805_2012Metric, symbol Device:C
- C2: footprint Capacitor_SMD:C_0805_2012Metric_Pad1.18x1.45mm_HandSolder -> Capacitor_SMD:C_0805_2012Metric
- R1, R2: footprint Resistor_SMD:R_0805_2012Metric_Pad1.20x1.40mm_HandSolder -> Resistor_SMD:R_0805_2012Metric
Connections:
- net ADC2_IO15 is gone; now on net B2: U1.8 (IO15)
- net LED_IO_35 is gone; now on net SCL: U1.29 (IO36)
- net +3V3: now also C1.1
- net A: now also U1.18 (IO10); no longer U1.20 (IO12)
- net B: now also U1.19 (IO11); no longer U1.22 (IO14)
- net B1: now also U1.6 (IO6); no longer U1.31 (IO38)
- net B2: no longer U1.21 (IO13)
- net BZ_PWM: now also U1.39 (IO1); no longer U1.38 (IO2)
- net C: now also U1.20 (IO12); no longer U1.19 (IO11)
- net CLK_75: now also U1.22 (IO14); no longer U1.11 (IO18)
- net D: now also U1.21 (IO13); no longer U1.18 (IO10)
- net EXP_SW_1: now also U1.31 (IO38); no longer U1.5 (IO5)
- net EXP_SW_2: now also U1.32 (IO39); no longer U1.6 (IO6)
- net EXP_SW_3: now also U1.33 (IO40); no longer U1.17 (IO9)
- net EXP_SW_4: now also U1.34 (IO41); no longer U1.39 (IO1)
- net EXP_SW_5: now also U1.9 (IO16); no longer U1.4 (IO4)
- net EXP_SW_6: now also U1.10 (IO17); no longer U1.12 (IO8)
- net EXP_SW_7: now also U1.11 (IO18); no longer U1.25 (IO48)
- net EXP_SW_8: now also U1.12 (IO8); no longer U1.24 (IO47)
- net G1: now also U1.4 (IO4); no longer U1.34 (IO41)
- net G2: now also U1.17 (IO9); no longer U1.32 (IO39)
- net GND: now also C1.2
- net LAT: now also U1.23 (IO21); no longer U1.10 (IO17)
- net MTH_SW: now also U1.30 (IO37); no longer U1.7 (IO7)
- net OE: now also U1.24 (IO47); no longer U1.9 (IO16)
- net R1: now also U1.5 (IO5); no longer U1.33 (IO40)
- net R2: now also U1.7 (IO7); no longer U1.30 (IO37)
- net SCL: no longer U1.23 (IO21)
- net UART_RX: now reaches U1.36 (IO44)
- net UART_TX: now reaches U1.37 (IO43)
- net IO42 renamed LED_IO_42
- new net FREE_IO: U1.25 (IO48)
- new net LED_IO_02: U1.38 (IO2)
- no-connect marks 5 -> 3

Commit message: final
Connections:
- net EXP_SW_1: now also U1.9 (IO16); no longer U1.31 (IO38)
- net EXP_SW_2: now also U1.10 (IO17); no longer U1.32 (IO39)
- net EXP_SW_3: now also U1.11 (IO18); no longer U1.33 (IO40)
- net EXP_SW_4: now also U1.12 (IO8); no longer U1.34 (IO41)
- net EXP_SW_5: now also U1.31 (IO38); no longer U1.9 (IO16)
- net EXP_SW_6: now also U1.32 (IO39); no longer U1.10 (IO17)
- net EXP_SW_7: now also U1.33 (IO40); no longer U1.11 (IO18)
- net EXP_SW_8: now also U1.34 (IO41); no longer U1.12 (IO8)
