File: PRTGN_v1/sub-sch/power.kicad_sch (KiCad schematic)
At the start: 20 parts, among them IC1 TPS565242DRLR, J2 Barrel_Jack, J3 Screw_Terminal_01x02, J4 Screw_Terminal_01x02, Q1 Q_PMOS, Q2 Q_PMOS, SW1 SW_DPDT_x2

Commit message: PCV updates
Parts:
- removed Q1: Q_PMOS, Package_TO_SOT_SMD:SOT-23-3, symbol Device:Q_PMOS_GSD
- removed R8: 10k, Resistor_SMD:R_0805_2012Metric_Pad1.20x1.40mm_HandSolder, symbol Device:R
- added C10, C3: 100nF, Capacitor_SMD:C_0805_2012Metric_Pad1.18x1.45mm_HandSolder, symbol Device:C
- added J1: USB_TypeC, sumec_brd:HRO_TYPE-C-31-M-12, symbol sumec_sch_lib:USB_TypeC
- added R3: 100k, Resistor_SMD:R_0805_2012Metric_Pad1.20x1.40mm_HandSolder, symbol Device:R
- added R6, R7: 15R, Resistor_SMD:R_0805_2012Metric_Pad1.20x1.40mm_HandSolder, symbol Device:R
- added U2: USBLC6-2SC6, Package_TO_SOT_SMD:TSOT-23-6_HandSoldering, symbol sumec_library:USBLC6-2SC6
- renumbered C3 to C4, C4 to C5, C5 to C6, C6 to C7, C7 to C8, C8 to C9, D5 to D1, D6 to D2, Q2 to Q1, R10 to R4, R11 to R5, R9 to R8
Connections:
- net VOUT is gone; now on net +5V: Q1.3 (D)
- net +5V: no longer D1.1 (K), D2.1 (K)
- net GND: now also C10.2, C3.1, J1.A1_B12 (GND), J1.B1_A12 (GND), R3.2, U2.2
- net VBATT: now also D1.2 (A); no longer Q1.2 (S), R8.1
- net VBUS 5V: now also C10.1, U2.5; no longer D2.2 (A)
- new net: D1.1 (K), D2.1 (K), Q1.2 (S), R8.1
- new net: R6.2, U2.1
- new net: R7.2, U2.3
- new net D+: U2.6
- new net D+ IN: J1.A6 (DP1), J1.B6 (DP2), R6.1
- new net D-: U2.4
- new net D- IN: J1.A7 (DN1), J1.B7 (DN2), R7.1
- new net SHLD: C3.2, J1.S1 (SHIELD), J1.S2 (SHIELD), J1.S3 (SHIELD), J1.S4 (SHIELD), R3.1
- new net VBUS_5V: D2.2 (A), J1.A4_B9 (VBUS), J1.B4_A9 (VBUS)
- no-connect marks 2 -> 6
Other:
- note added: "CONN / TERMINALS"
- note added: "ESD PROTECTION"
- note added: "GPIO USB 20 D+ (green) 19 D- (white) GND GND (black) VBUS +5V (red)"
- note added: "HIGH SIDE"
- note added: "USB CONNECTOR"
- note added: "USB Type-C Connector Data transfer USB connector connected to ESP32 using CDC method"
- note added: "USB-C"
- note removed: "5V TERMINAL"
- note removed: "BARREL JACK"
- note removed: "Power switching between 5V VBUS - USB and 5V Buck converter - BATT"
- note removed: "SWITCHING SIMULATION - FALSTAD"
- note removed: "USB POWER SWITCH"
- moved on the sheet: C4, C5, C6, C7, C8, C9, D1, D2, IC1, J2, J3, J4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

Commit message: PCB
Parts:
- added J10, J11: JST-VH4, Connector_JST:JST_VH_B4P-VH-B_1x04_P3.96mm_Vertical, symbol Connector:Conn_01x04_Pin
Connections:
- net +5V: now also J10.1 (Pin_1), J10.2 (Pin_2), J11.1 (Pin_1), J11.2 (Pin_2)
- net GND: now also J10.3 (Pin_3), J10.4 (Pin_4), J11.3 (Pin_3), J11.4 (Pin_4)

Commit message: layout PCB etc
Connections:
- net VBUS 5V is gone; now on net VBUS_5V: C10.1, U2.5
Changed lines of the file:
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@@
 		)
 	)
-	(global_label "VBUS 5V"
+	(global_label "VBUS_5V"
 		(shape input)
 		(at 173.99 64.77 0)
@@
 		)
 		(property "Intersheetrefs" "${INTERSHEET_REFS}"
-			(at 182.7064 64.77 0)
+			(at 181.8219 64.77 0)
 			(effects
 				(font

Commit message: pcb silksdnree neded
Parts:
- removed J2: Barrel_Jack, Connector_BarrelJack:BarrelJack_Horizontal, symbol Connector:Barrel_Jack_MountingPin
- removed SW1: SW_DPDT_x2, sumec_brd:Custom_SPDT_2.5_Switch, symbol Switch:SW_DPDT_x2
- added J3, J4: SOLDER PAD, PRTGN_brd:SolderWirePad_1x01_SMD, symbol Connector:Conn_01x01_Pin
- added SW1: SW_SPDT, sumec_brd:Custom_SPDT_2.5_Switch, symbol Switch:SW_SPDT
- C10, C3, C5, C9: footprint Capacitor_SMD:C_0805_2012Metric_Pad1.18x1.45mm_HandSolder -> Capacitor_SMD:C_0805_2012Metric
- C4, C6, C7, C8: footprint Capacitor_Tantalum_SMD:CP_EIA-2012-12_Kemet-R_Pad1.30x1.05mm_HandSolder -> Capacitor_Tantalum_SMD:CP_EIA-2012-12_Kemet-R
- D1, D2: footprint Diode_SMD:D_1206_3216Metric_Pad1.42x1.75mm_HandSolder -> Diode_SMD:D_2114_3652Metric
- J6: renamed from J3; footprint TerminalBlock:TerminalBlock_Xinya_XY308-2.54-2P_1x02_P2.54mm_Horizontal -> TerminalBlock_Phoenix:TerminalBlock_Phoenix_MKDS-1,5-2-5.08_1x02_P5.08mm_Horizontal
- J7: renamed from J4; footprint TerminalBlock:TerminalBlock_Xinya_XY308-2.54-2P_1x02_P2.54mm_Horizontal -> TerminalBlock_Phoenix:TerminalBlock_Phoenix_MKDS-1,5-2-5.08_1x02_P5.08mm_Horizontal
- R3, R4, R5, R6, R7, R8: footprint Resistor_SMD:R_0805_2012Metric_Pad1.20x1.40mm_HandSolder -> Resistor_SMD:R_0805_2012Metric
- U2: footprint Package_TO_SOT_SMD:TSOT-23-6_HandSoldering -> Package_TO_SOT_SMD:TSOT-23-6
- renumbered J10 to J2, J11 to J5
Connections:
- net FET_SW: now also SW1.1 (A)
- net GND: now also J4.1 (Pin_1), SW1.2 (B)
- net VBATT: now also J3.1 (Pin_1)
- no-connect marks 6 -> 5
Other:
- moved on the sheet: J2, J5

Commit message: didnt close it
Connections:
- net D+: now also U2.4; no longer U2.6
- net D-: now also U2.6; no longer U2.4
- net at U2.1: now also R7.2; no longer R6.2
- net at U2.3: now also R6.2; no longer R7.2
Other:
- moved on the sheet: R6, R7
Changed lines of the file:
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@@
 	(wire
 		(pts
+			(xy 120.65 52.07) (xy 121.92 52.07)
+		)
+		(stroke
+			(width 0)
+			(type default)
+		)
+	)
+	(wire
+		(pts
 			(xy 245.11 69.85) (xy 246.38 69.85)
 		)
@@
 	(wire
 		(pts
-			(xy 120.65 52.07) (xy 121.92 52.07)
-		)
-		(stroke
-			(width 0)
-			(type default)
-		)
-	)
-	(wire
-		(pts
 			(xy 85.09 124.46) (xy 86.36 124.46)
 		)
@@
 	(wire
 		(pts
-			(xy 120.65 77.47) (xy 121.92 77.47)
+			(xy 129.54 64.77) (xy 130.81 64.77)
 		)
 		(stroke
@@
 	(wire
 		(pts
-			(xy 129.54 64.77) (xy 130.81 64.77)
+			(xy 245.11 58.42) (xy 246.38 58.42)
 		)
 		(stroke
@@
 	(wire
 		(pts
-			(xy 245.11 58.42) (xy 246.38 58.42)
+			(xy 120.65 77.47) (xy 121.92 77.47)
 		)
 		(stroke
@@
 		)
 	)
-	(global_label "VBUS_5V"
+	(global_label "D- IN"
 		(shape input)
-		(at 254 104.14 0)
+		(at 120.65 52.07 180)
 		(fields_autoplaced yes)
 		(effects
@@
 				(color 0 0 0 1)
 			)
-			(justify left)
+			(justify right)
 		)
 		(property "Intersheetrefs" "${INTERSHEET_REFS}"
-			(at 261.8319 104.14 0)
+			(at 113.8383 52.07 0)
 			(effects
 				(font
 					(size 1.27 1.27)
 				)
-				(justify left)
+				(justify right)
 				(hide yes)
 			)
 		)
 	)
-	(global_label "D- IN"
+	(global_label "VBUS_5V"
 		(shape input)
-		(at 120.65 77.47 180)
+		(at 254 104.14 0)
 		(fields_autoplaced yes)
 		(effects
@@
 				(color 0 0 0 1)
 			)
-			(justify right)
+			(justify left)
 		)
 		(property "Intersheetrefs" "${INTERSHEET_REFS}"
-			(at 113.8383 77.47 0)
+			(at 261.8319 104.14 0)
 			(effects
 				(font
 					(size 1.27 1.27)
 				)
-				(justify right)
+				(justify left)
 				(hide yes)
 			)
@@
 		)
 	)
-	(global_label "FB"
-		(shape input)
-		(at 85.09 118.11 180)
+	(global_label "D-"
+		(shape output)
+		(at 172.72 52.07 0)
 		(fields_autoplaced yes)
 		(effects
@@
 				(color 0 0 0 1)
 			)
-			(justify right)
+			(justify left)
 		)
 		(property "Intersheetrefs" "${INTERSHEET_REFS}"
-			(at 81.2148 118.11 0)
+			(at 176.4848 52.07 0)
 			(effects
 				(font
 					(size 1.27 1.27)
 				)
-				(justify right)
+				(justify left)
 				(hide yes)
 			)
 		)
 	)
-	(global_label "D+ IN"
-		(shape input)
-		(at 81.28 66.04 180)
+	(global_label "D+"
+		(shape output)
+		(at 172.72 77.47 0)
 		(fields_autoplaced yes)
 		(effects
@@
 				(color 0 0 0 1)
 			)
-			(justify right)
+			(justify left)
 		)
 		(property "Intersheetrefs" "${INTERSHEET_REFS}"
-			(at 75.7068 66.04 0)
+			(at 176.5532 77.47 0)
 			(effects
 				(font
 					(size 1.27 1.27)
 				)
-				(justify right)
+				(justify left)
 				(hide yes)
 			)
 		)
 	)
-	(global_label "D+ IN"
+	(global_label "FB"
 		(shape input)
-		(at 119.38 63.5 0)
+		(at 85.09 118.11 180)
 		(fields_autoplaced yes)
 		(effects
@@
 				(color 0 0 0 1)
 			)
-			(justify left)
+			(justify right)
 		)
 		(property "Intersheetrefs" "${INTERSHEET_REFS}"
-			(at 124.9532 63.5 0)
+			(at 81.2148 118.11 0)
 			(effects
 				(font
 					(size 1.27 1.27)
 				)
-				(justify left)
+				(justify right)
 				(hide yes)
 			)
 		)
 	)
-	(global_label "D+"
-		(shape output)
-		(at 172.72 52.07 0)
+	(global_label "D+ IN"
+		(shape input)
+		(at 81.28 66.04 180)
 		(fields_autoplaced yes)
 		(effects
@@
 				(color 0 0 0 1)
 			)
-			(justify left)
+			(justify right)
 		)
 		(property "Intersheetrefs" "${INTERSHEET_REFS}"
-			(at 176.5532 52.07 0)
+			(at 75.7068 66.04 0)
 			(effects
 				(font
 					(size 1.27 1.27)
 				)
-				(justify left)
+				(justify right)
 				(hide yes)
 			)
 		)
 	)
-	(global_label "D-"
-		(shape output)
-		(at 172.72 77.47 0)
+	(global_label "D+ IN"
+		(shape input)
+		(at 120.65 77.47 180)
 		(fields_autoplaced yes)
 		(effects
@@
 				(color 0 0 0 1)
 			)
-			(justify left)
+			(justify right)
 		)
 		(property "Intersheetrefs" "${INTERSHEET_REFS}"
-			(at 176.4848 77.47 0)
+			(at 113.8383 77.47 0)
 			(effects
 				(font
 					(size 1.27 1.27)
 				)
-				(justify left)
+				(justify right)
 				(hide yes)
 			)
@@
 	(global_label "D+ IN"
 		(shape input)
-		(at 120.65 52.07 180)
+		(at 119.38 63.5 0)
 		(fields_autoplaced yes)
 		(effects
@@
 				(color 0 0 0 1)
 			)
-			(justify right)
+			(justify left)
 		)
 		(property "Intersheetrefs" "${INTERSHEET_REFS}"
-			(at 113.8383 52.07 0)
+			(at 124.9532 63.5 0)
 			(effects
 				(font
 					(size 1.27 1.27)
 				)
-				(justify right)
+				(justify left)
 				(hide yes)
 			)
@@
 	(symbol
 		(lib_id "Device:R")
-		(at 125.73 77.47 90)
+		(at 125.73 52.07 90)
 		(unit 1)
 		(exclude_from_sim no)
@@
 		(dnp no)
 		(property "Reference" "R7"
-			(at 123.825 73.025 90)
+			(at 123.825 47.625 90)
 			(effects
 				(font
@@
 		)
 		(property "Value" "15R"
-			(at 123.825 74.93 90)
+			(at 123.825 49.53 90)
 			(effects
 				(font
@@
 		)
 		(property "Footprint" "Resistor_SMD:R_0805_2012Metric"
-			(at 125.73 79.248 90)
+			(at 125.73 53.848 90)
 			(effects
 				(font
@@
 		)
 		(property "Datasheet" "~"
-			(at 125.73 77.47 0)
+			(at 125.73 52.07 0)
 			(effects
 				(font
@@
 		)
 		(property "Description" ""
-			(at 125.73 77.47 0)
+			(at 125.73 52.07 0)
 			(effects
 				(font
@@
 	(symbol
 		(lib_id "Device:R")
-		(at 125.73 52.07 90)
+		(at 125.73 77.47 90)
 		(unit 1)
 		(exclude_from_sim no)
@@
 		(dnp no)
 		(property "Reference" "R6"
-			(at 123.825 47.625 90)
+			(at 123.825 73.025 90)
 			(effects
 				(font
@@
 		)
 		(property "Value" "15R"
-			(at 123.825 49.53 90)
+			(at 123.825 74.93 90)
 			(effects
 				(font
@@
 		)
 		(property "Footprint" "Resistor_SMD:R_0805_2012Metric"
-			(at 125.73 53.848 90)
+			(at 125.73 79.248 90)
 			(effects
 				(font
@@
 		)
 		(property "Datasheet" "~"
-			(at 125.73 52.07 0)
+			(at 125.73 77.47 0)
 			(effects
 				(font
@@
 		)
 		(property "Description" ""
-			(at 125.73 52.07 0)
+			(at 125.73 77.47 0)
 			(effects
 				(font
