File: Electronics/PRTGN_v1/sub-sch/power.kicad_sch (KiCad schematic)
At the start: 28 parts, among them IC1 TPS565242DRLR, J1 USB_TypeC, J2 JST-VH4, J3 SOLDER PAD, J4 SOLDER PAD, J5 JST-VH4, J6 Screw_Terminal_01x02, J7 Screw_Terminal_01x02, Q1 Q_PMOS, SW1 SW_SPDT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

Commit message: new code
Parts:
- U2: DESCRIPTION 17V Clamp 5A (8/20µs) Ipp Tvs Diode Surface Mount SOT-23-6 -> (none)
